File: Bimasakti BM-13 EVO/Power Delivery management/Power Delivery Management_3.3V/Power Delivery Management_3.3V.kicad_pcb (KiCad board)
At the start: 2 copper layers, 42.4 x 42.4 mm, 24 parts, among them J1 +12V In, J2 Conn_01x03_Socket, J3 Slow Start

Commit message: tambah led
Parts:
- added D2: LED, LED_SMD:LED_0603_1608Metric_Pad1.05x0.95mm_HandSolder, F.Cu at (44.3, 46.9)
- added R5: 1k, Resistor_SMD:R_0603_1608Metric, F.Cu at (42.8, 46.8)
- added R6: 1.5k, Resistor_SMD:R_0603_1608Metric, F.Cu at (45.8, 46.8)
Routing:
- net +5v: track 0.00 -> 96.7 mm, vias 0 -> 2
- net (no net): track 213.6 -> 118.7 mm, vias 61 -> 59
- net Net-(D2-A): track 0.00 -> 3.81 mm
