File: Bimasakti BM-13 EVO/Power Delivery management/Power Delivery Management_3.3V/Power Delivery Management_3.3V.kicad_sch (KiCad schematic)
At the start: 24 parts, among them J1 +12V In, J2 Slow Start, J3 Conn_01x03_Socket

Commit message: tambah led
Parts:
- added D2: LED, LED_SMD:LED_0603_1608Metric_Pad1.05x0.95mm_HandSolder, symbol Device:LED
- added R5: 1k, Resistor_SMD:R_0603_1608Metric, symbol Device:R
- added R6: 1.5k, Resistor_SMD:R_0603_1608Metric, symbol Device:R
Connections:
- net GND: now also D2.1 (K), R6.1
- new net: D2.2 (A), R5.2, R6.2
- new net +5v: R5.1
