File: Bimasakti BM-13 EVO/Telemetry/Telemetry TAZ V1/Telemetry TAZ V1.kicad_sch (KiCad schematic)
At the start: 12 parts, among them J1 Screw_Terminal_01x04, J12 POWER, J2 Conn_02x05_Odd_Even, J6 Screw_Terminal_01x04, J7 Screw_Terminal_01x03, U1 ESP32-DEVKIT-V1

Commit message: tambah led
Parts:
- added R1: R, symbol Device:R
Changed lines of the file:
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@@
+	)
+	(symbol
+		(lib_id "Device:R")
+		(at 85.09 87.63 0)
+		(unit 1)
+		(exclude_from_sim no)
+		(in_bom yes)
+		(on_board yes)
+		(dnp no)
+		(fields_autoplaced yes)
+		(property "Reference" "R1"
+			(at 87.63 86.3599 0)
+			(effects
+				(font
+					(size 1.27 1.27)
+				)
+				(justify left)
+			)
+		)
+		(property "Value" "R"
+			(at 87.63 88.8999 0)
+			(effects
+				(font
+					(size 1.27 1.27)
+				)
+				(justify left)
+			)
+		)
+		(property "Footprint" ""
+			(at 83.312 87.63 90)
+			(effects
+				(font
+					(size 1.27 1.27)
+				)
+				(hide yes)
+			)
+		)
+		(property "Datasheet" "~"
+			(at 85.09 87.63 0)
+			(effects
+				(font
+					(size 1.27 1.27)
+				)
+				(hide yes)
+			)
+		)
+		(property "Description" "Resistor"
+			(at 85.09 87.63 0)
+			(effects
+				(font
+					(size 1.27 1.27)
+				)
+				(hide yes)
+			)
+		)
+		(pin "2"
+		)
+		(pin "1"
+		)
+		(instances
+			(project ""
+				(path "/f434244f-15a7-4de2-9e24-274a2aea42b1"
+					(reference "R1")
+					(unit 1)
+				)
+			)
+		)
 	)
 	(symbol
