File: Bimasakti BM-13 EVO/Vehicle Control Unit/VCU.kicad_sch (KiCad schematic)
At the start: 12 parts, among them J1 Conn_01x02_Socket, J2 Conn_01x02_Socket, T1 AOD4189, U1 MCP2551-I-SN

Commit message: add footprint library to project
Changed lines of the file:
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@@
 (kicad_sch
-	(version 20231120)
+	(version 20250114)
 	(generator "eeschema")
-	(generator_version "8.0")
+	(generator_version "9.0")
 	(paper "A4")
+	(rectangle
+		(start 143.51 80.01)
+		(end 143.51 80.01)
+		(stroke
+			(width 0)
+			(type default)
+		)
+		(fill
+			(type none)
+		)
+	)
 	(junction
 		(at 71.12 118.11)
@@
 			(width 0)
 			(type default)
-		)
-	)
-	(rectangle
-		(start 143.51 80.01)
-		(end 143.51 80.01)
-		(stroke
-			(width 0)
-			(type default)
-		)
-		(fill
-			(type none)
 		)
 	)
@@
 		)
 	)
+	(embedded_fonts no)
 )

Commit message: Revert "add footprint library to project"
This reverts commit c2ea81f1652adadaa2769e08c07f448226fedb71.
Changed lines of the file:
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@@
 (kicad_sch
-	(version 20250114)
+	(version 20231120)
 	(generator "eeschema")
-	(generator_version "9.0")
+	(generator_version "8.0")
 	(paper "A4")
-	(rectangle
-		(start 143.51 80.01)
-		(end 143.51 80.01)
-		(stroke
-			(width 0)
-			(type default)
-		)
-		(fill
-			(type none)
-		)
-	)
 	(junction
 		(at 71.12 118.11)
@@
 			(width 0)
 			(type default)
+		)
+	)
+	(rectangle
+		(start 143.51 80.01)
+		(end 143.51 80.01)
+		(stroke
+			(width 0)
+			(type default)
+		)
+		(fill
+			(type none)
 		)
 	)
@@
 		)
 	)
-	(embedded_fonts no)
 )
