File: Bimasakti BM-13 EVO/Power Delivery management/PDM Motherboard/PDM MOTHERBOARD/PDM MOTHERBOARD.kicad_sch (KiCad schematic)
At the start: 4 parts

Commit message: progress on motherboard pdm
Parts:
- added F2: Fuse, Fuse:Fuseholder_Clip-5x20mm_Bel_FC-203-22_Lateral_P17.80x5.00mm_D1.17mm_Horizontal, symbol Device:Fuse
- added U2: ~, Library:SOIC-8 (AOD), symbol New_Library:AOD4407
- added keluar2, masuk2: ~, Connector_JST:JST_EH_B2B-EH-A_1x02_P2.50mm_Vertical, symbol Connector:Conn_01x02_Socket
- renumbered +12Vin to keluar1, +12V to masuk1
Connections:
- net GND: now also F2.2, U2.2 (G), keluar2.2 (Pin_2)
- new net: U2.3 (S), keluar2.1 (Pin_1)
- new net: F2.1, masuk2.1 (Pin_1)
- new net: U2.1 (D), masuk2.2 (Pin_2)
