File: Bimasakti BM-13 EVO/Power Delivery management/PDM Motherboard/PDM MOTHERBOARD.kicad_pcb (KiCad board)
At the start: 2 copper layers, 78.2 x 101.3 mm, 24 parts

Commit message: update motherboard pdm selesai
Parts:
- removed 5Vin2, 5Vin3, 5Vin4: ~, Connector_JST:JST_EH_B2B-EH-A_1x02_P2.50mm_Vertical
- removed D3: SMAJ5.0A, Diode_SMD:D_SMA
- added 3Vin1: ~, Connector_JST:JST_EH_B2B-EH-A_1x02_P2.50mm_Vertical, F.Cu at (113.7, 59.4)
- added 5out3: ~, Connector_JST:JST_EH_B2B-EH-A_1x02_P2.50mm_Vertical, F.Cu at (151.5, 106.0)
- added 5out4: ~, Connector_JST:JST_EH_B2B-EH-A_1x02_P2.50mm_Vertical, F.Cu at (151.5, 85.6)
- added F4: 1A, Fuse:Fuseholder_Cylinder-5x20mm_Schurter_0031_8201_Horizontal_Open, F.Cu at (123.4, 104.5)
- added F7: 1A, Fuse:Fuseholder_Cylinder-5x20mm_Schurter_0031_8201_Horizontal_Open, F.Cu at (123.4, 82.9)
- F1, F10, F3, F5, F6, F8: footprint Fuse:Fuseholder_Clip-5x20mm_Bel_FC-203-22_Lateral_P17.80x5.00mm_D1.17mm_Horizontal -> Fuse:Fuseholder_Cylinder-5x20mm_Schurter_0031_8201_Horizontal_Open
- U1: footprint Library:SOIC-8 (AOD) -> AO4407A:SOIC-8 (AOD)
- moved D1 88.5 mm to (79.2, 47.2), turned to -90 degrees
- moved D4 66.6 mm to (119.1, 96.2), turned to -90 degrees
- moved D6 58.7 mm to (117.5, 29.1), turned to -90 degrees
- moved F3 56.5 mm to (123.4, 94.1)
- moved F10 53.2 mm to (123.0, 26.7)
- moved D5 49.1 mm to (118.6, 59.1), turned to -90 degrees
- moved 5Vin1 42.0 mm to (114.2, 96.4), turned to 90 degrees
- moved F1 29.8 mm to (58.9, 59.7)
- moved F5 29.7 mm to (123.4, 72.1)
- moved F6 23.1 mm to (123.2, 46.2)
- moved F8 22.2 mm to (123.2, 56.9)
- moved 12vout1 21.2 mm to (151.0, 29.1), turned to 90 degrees
- moved 5out2 19.4 mm to (151.5, 97.0), turned to 90 degrees
- moved 5out1 19.1 mm to (151.3, 74.6), turned to 90 degrees
- moved 3v3out2 18.0 mm to (151.0, 59.4), turned to 90 degrees
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Connections:
- 3v3out1 pad 2: Net-(3v3out1-Pin_2) -> GND
- 3v3out2 pad 2: Net-(3v3out2-Pin_2) -> GND
- 5Vin1 pad 1: Net-(5Vin1-Pin_1) -> GND
- 5Vin1 pad 2: Net-(5Vin1-Pin_2) -> 5Vin
- 5out1 pad 2: Net-(5Vin1-Pin_1) -> GND
- 5out2 pad 2: Net-(5Vin4-Pin_1) -> GND
- D4 pad 1: Net-(5Vin1-Pin_2) -> 5Vin
- D4 pad 2: Net-(5Vin1-Pin_1) -> GND
- D5 pad 1: Net-(5Vin2-Pin_2) -> 3Vin
- D5 pad 2: Net-(3v3out1-Pin_2) -> GND
- D6 pad 1: Net-(5Vin3-Pin_2) -> +12
- D6 pad 2: Net-(3v3out2-Pin_2) -> GND
- F3 pad 1: Net-(5Vin4-Pin_2) -> 5Vin
- F5 pad 1: Net-(5Vin1-Pin_2) -> 5Vin
- F6 pad 1: Net-(5Vin2-Pin_2) -> 3Vin
- F8 pad 1: Net-(5Vin3-Pin_2) -> 3Vin
Routing:
- net +12: track 24.2 -> 93.0 mm
- net 5Vin: track 0.00 -> 41.0 mm
- net Net-(12in1-Pin_1): track 11.7 -> 38.6 mm
- net GND: track 24.4 -> 51.3 mm
- net 3Vin: track 0.00 -> 20.3 mm
- net Net-(12in1-Pin_2): track 37.6 -> 51.5 mm
- net Net-(5out2-Pin_1): track 0.00 -> 6.80 mm
- net Net-(5out4-Pin_1): track 0.00 -> 6.69 mm
- net Net-(12vout1-Pin_1): track 0.00 -> 6.48 mm
- net Net-(3v3out1-Pin_1): track 0.00 -> 6.44 mm
- net Net-(5out1-Pin_1): track 0.00 -> 6.42 mm
- net Net-(3v3out2-Pin_1): track 0.00 -> 6.30 mm
- net Net-(5out3-Pin_1): track 0.00 -> 6.29 mm
- added copper zone on B.Cu, net GND
- added copper zone on F.Cu, net GND
Other:
- board size 78.2 x 101.3 mm -> 108 x 101.3 mm
