File: Bimasakti BM-13 EVO/PCB/Power Delivery management/Power Delivery Management_5V/Power Delivery Management_5V.kicad_sch (KiCad schematic)
At the start: 27 parts, among them J1 +12V In, J2 Conn_01x03_Socket, J3 Slow Start

Commit message: pdm
Parts:
- L1: value 12uH -> 4.7uH
- R3: value 1.5k -> 3k
- R4: value 390 -> 220
Connections:
- net +12V: now also J1.1 (Pin_1)
- net GND: now also J1.2 (Pin_2)
Changed lines of the file:
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@@
+	(wire
+		(pts
+			(xy 29.21 40.64) (xy 30.48 40.64)
+		)
+		(stroke
+			(width 0)
+			(type default)
+		)
+	)
 	(wire
 		(pts
@@
 		(pts
 			(xy 87.63 25.4) (xy 88.9 25.4)
+		)
+		(stroke
+			(width 0)
+			(type default)
+		)
+	)
+	(wire
+		(pts
+			(xy 29.21 38.1) (xy 30.48 38.1)
 		)
 		(stroke
@@
 			)
 		)
-		(property "Value" "390"
+		(property "Value" "220"
 			(at 118.364 50.8 90)
 			(effects
@@
 		(property "Description" "Resistor"
 			(at 118.11 48.26 0)
+			(effects
+				(font
+					(size 1.27 1.27)
+				)
+				(hide yes)
+			)
+		)
+		(property "Field5" ""
+			(at 118.11 48.26 90)
 			(effects
 				(font
@@
 			)
 		)
-		(property "Value" "12uH"
+		(property "Value" "4.7uH"
 			(at 124.46 29.21 90)
 			(effects
@@
 			)
 		)
-		(property "Value" "1.5k"
+		(property "Value" "3k"
 			(at 128.27 50.546 90)
 			(effects
