File: Bimasakti BM-13 EVO/PCB/Telemetry V.3 BM13 EVO Hy/Telemetry V.3 BM13 EVO Hy.kicad_pcb (KiCad board)
At the start: 2 copper layers, 86 x 70 mm, 28 parts, among them J1 MSD-4-A, J2 CON INT/32, J4 Conn_01x04_Socket, U1 ESP32-DEVKIT-V1, U2 74LVC125APW_118, U3 DS3231SN_

Commit message: Aku Wheelspeed
Routing:
- net /CS: track 12.1 -> 10.8 mm
- net /SCK: track 12.6 -> 11.4 mm
- net /RX: track 20.2 -> 19.2 mm
- net +3.3V: track 91.8 -> 90.9 mm
- net GND: track 30.7 -> 30.8 mm, vias 7 -> 43
