File: Bimasakti BM-13 EVO/PCB/Wheelspeed Module/Wheelspeed Module/Wheelspeed Module.kicad_pcb (KiCad board)
At the start: 2 copper layers, 53 x 64 mm, 31 parts, among them J1 Conn_01x20_Pin, J2 Conn_01x20_Pin, U1 esp32-wemos-d1-mini, U2 LM393, U3 LM393

Commit message: Aku VCU
Parts:
- added U4: ESP32-C3_SUPERMINI_TH, ESP32 Supermini:MODULE_ESP32-C3_SUPERMINI, F.Cu at (9.28, 12.9)
Connections:
- J1 pad 14: unconnected-(J1-Pin_14-Pad14) -> GND
- J1 pad 15: unconnected-(J1-Pin_15-Pad15) -> GND
- J1 pad 16: unconnected-(J1-Pin_16-Pad16) -> GND
- J1 pad 4: unconnected-(J1-Pin_4-Pad4) -> GND
- J1 pad 5: unconnected-(J1-Pin_5-Pad5) -> GND
- J2 pad 6: unconnected-(J2-Pin_6-Pad6) -> GND
- J2 pad 7: unconnected-(J2-Pin_7-Pad7) -> GND
- J2 pad 8: unconnected-(J2-Pin_8-Pad8) -> GND
- J2 pad 9: unconnected-(J2-Pin_9-Pad9) -> GND
