File: Bimasakti BM-13 EVO/PCB/Wheelspeed Module/Wheelspeed Module/Wheelspeed Module.kicad_sch (KiCad schematic)
At the start: 14 parts, among them U1 LM339, U5 ESP32-DEVKIT-V1

Commit message: Aku Wheelspeed
Parts:
- removed U1: LM339, symbol Comparator:LM339
- removed U5: ESP32-DEVKIT-V1, ESP32-DEVKIT-V1:MODULE_ESP32_DEVKIT_V1, symbol ESP32-DEVKIT-V1:ESP32-DEVKIT-V1
- added C1, C2: C_Small, Capacitor_SMD:C_0603_1608Metric_Pad1.08x0.95mm_HandSolder, symbol Device:C_Small
- added FL1, FL2, FR1, FR2, RL1, RL2, RR1, RR2: TestPoint, TestPoint:TestPoint_Bridge_Pitch2.54mm_Drill0.7mm, symbol Connector:TestPoint
- added J1, J2: Conn_01x20_Pin, Connector_PinHeader_2.54mm:PinHeader_1x20_P2.54mm_Vertical, symbol Connector:Conn_01x20_Pin
- added R13, R14, R15, R16: 400, Resistor_SMD:R_0603_1608Metric_Pad0.98x0.95mm_HandSolder, symbol Device:R_Small_US
- added U1: esp32-wemos-d1-mini, kicad-esp32-wemos-d1-mini-master:esp32-wemos-d1-mini, symbol esp32-wemos-d1-mini:esp32-wemos-d1-mini
- added U2, U3: LM393, LM393:SO8_STM, symbol Comparator:LM393
- R1, R3, R5, R7: value R_Small_US -> 10K; footprint (none) -> Resistor_SMD:R_0603_1608Metric_Pad0.98x0.95mm_HandSolder
- R10, R11, R12, R9: value R_Small_US -> 1K; footprint (none) -> Resistor_SMD:R_0603_1608Metric_Pad0.98x0.95mm_HandSolder
- R2: value R_Small_US -> 22K; footprint (none) -> Resistor_SMD:R_0603_1608Metric_Pad0.98x0.95mm_HandSolder
- R4, R6, R8: value R_Small_US -> 20K; footprint (none) -> Resistor_SMD:R_0603_1608Metric_Pad0.98x0.95mm_HandSolder
Connections:
- net +12V: now also C1.1, C2.1, J1.2 (Pin_2), R13.1, R14.1, R15.1, R16.1, U2.8 (V+), U3.8 (V+)
- net GND: now also C1.2, C2.2, J1.3 (Pin_3), J2.5 (Pin_5), U1.1 (GND), U1.22 (GND), U1.33 (GND), U2.4 (V-), U3.4 (V-)
- net at R1.2, R2.1: now also U2.2 (-)
- net at R5.2, R6.1: now also U3.2 (-)
- net +3.3V: now reaches R9.1
- net +3.3V: now also R10.1, R11.1, R12.1, U1.16 (3V3)
- net WS_FR_Signal: now reaches R9.2
- net WS_FR_Signal: now also FR2.1, U1.25 (IO_22/D1/SCL), U2.1
- net WS_RR_Signal: now reaches R11.2
- net WS_RR_Signal: now also RR2.1, U1.29 (IO_17/D3), U3.1
- net at R7.2, R8.1: now also U3.6 (-)
- net at R3.2, R4.1: now also U2.6 (-)
- net WS_FL_Signal: now reaches R10.2
- net WS_FL_Signal: now also FL2.1, U1.27 (IO_21/D2/SDA), U2.7
- net WS_RL_Signal: now reaches R12.2
- net WS_RL_Signal: now also RL2.1, U1.31 (IO_16/D4), U3.7
- new net +5V: J1.1 (Pin_1), U1.35 (VCC_(USB))
- new net CS: J2.4 (Pin_4), U1.14 (IO_05/D8)
- new net MISO: J2.2 (Pin_2), U1.10 (IO_19/D6)
- new net MOSI: J2.3 (Pin_3), U1.12 (IO_23/D7)
- new net SCK: J2.1 (Pin_1), U1.8 (IO_18/D5)
- new net WS_FL: FL1.1, J1.18 (Pin_18), R14.2, U2.5 (+)
- new net WS_FR: FR1.1, J1.17 (Pin_17), R13.2, U2.3 (+)
- new net WS_RL: J1.20 (Pin_20), R16.2, RL1.1, U3.5 (+)
- new net WS_RR: J1.19 (Pin_19), R15.2, RR1.1, U3.3 (+)
Other:
- moved on the sheet: R1, R10, R11, R12, R2, R3, R4, R5, R6, R7, R8, R9

Commit message: Aku Telemetry
Parts:
- added U4: ESP32-C3_SUPERMINI_TH, ESP32 Supermini:MODULE_ESP32-C3_SUPERMINI, symbol ESP32-C3_SUPERMINI_TH:ESP32-C3_SUPERMINI_TH
Changed lines of the file:
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@@
+	)
+	(symbol
+		(lib_id "ESP32-C3_SUPERMINI_TH:ESP32-C3_SUPERMINI_TH")
+		(at 69.85 130.81 0)
+		(unit 1)
+		(exclude_from_sim no)
+		(in_bom yes)
+		(on_board yes)
+		(dnp no)
+		(fields_autoplaced yes)
+		(property "Reference" "U4"
+			(at 69.85 110.49 0)
+			(effects
+				(font
+					(size 1.27 1.27)
+				)
+			)
+		)
+		(property "Value" "ESP32-C3_SUPERMINI_TH"
+			(at 69.85 113.03 0)
+			(effects
+				(font
+					(size 1.27 1.27)
+				)
+			)
+		)
+		(property "Footprint" "ESP32 Supermini:MODULE_ESP32-C3_SUPERMINI"
+			(at 69.85 130.81 0)
+			(effects
+				(font
+					(size 1.27 1.27)
+				)
+				(justify bottom)
+				(hide yes)
+			)
+		)
+		(property "Datasheet" ""
+			(at 69.85 130.81 0)
+			(effects
+				(font
+					(size 1.27 1.27)
+				)
+				(hide yes)
+			)
+		)
+		(property "Description" ""
+			(at 69.85 130.81 0)
+			(effects
+				(font
+					(size 1.27 1.27)
+				)
+				(hide yes)
+			)
+		)
+		(property "MF" "Espressif Systems"
+			(at 69.85 130.81 0)
+			(effects
+				(font
+					(size 1.27 1.27)
+				)
+				(justify bottom)
+				(hide yes)
+			)
+		)
+		(property "MAXIMUM_PACKAGE_HEIGHT" "4.2mm"
+			(at 69.85 130.81 0)
+			(effects
+				(font
+					(size 1.27 1.27)
+				)
+				(justify bottom)
+				(hide yes)
+			)
+		)
+		(property "Package" "Package"
+			(at 69.85 130.81 0)
+			(effects
+				(font
+					(size 1.27 1.27)
+				)
+				(justify bottom)
+				(hide yes)
+			)
+		)
+		(property "Price" "None"
+			(at 69.85 130.81 0)
+			(effects
+				(font
+					(size 1.27 1.27)
+				)
+				(justify bottom)
+				(hide yes)
+			)
+		)
+		(property "Check_prices" "https://www.snapeda.com/parts/ESP32-C3%20SuperMini_TH/Espressif+Systems/view-part/?ref=eda"
+			(at 69.85 130.81 0)
+			(effects
+				(font
+					(size 1.27 1.27)
+				)
+				(justify bottom)
+				(hide yes)
+			)
+		)
+		(property "STANDARD" "Manufacturer Recommendations"
+			(at 69.85 130.81 0)
+			(effects
+				(font
+					(size 1.27 1.27)
+				)
+				(justify bottom)
+				(hide yes)
+			)
+		)
+		(property "PARTREV" ""
+			(at 69.85 130.81 0)
+			(effects
+				(font
+					(size 1.27 1.27)
+				)
+				(justify bottom)
+				(hide yes)
+			)
+		)
+		(property "SnapEDA_Link" "https://www.snapeda.com/parts/ESP32-C3%20SuperMini_TH/Espressif+Systems/view-part/?ref=snap"
+			(at 69.85 130.81 0)
+			(effects
+				(font
+					(size 1.27 1.27)
+				)
+				(justify bottom)
+				(hide yes)
+			)
+		)
+		(property "MP" "ESP32-C3 SuperMini_TH"
+			(at 69.85 130.81 0)
+			(effects
+				(font
+					(size 1.27 1.27)
+				)
+				(justify bottom)
+				(hide yes)
+			)
+		)
+		(property "Description_1" "Super tiny ESP32-C3 board"
+			(at 69.85 130.81 0)
+			(effects
+				(font
+					(size 1.27 1.27)
+				)
+				(justify bottom)
+				(hide yes)
+			)
+		)
+		(property "Availability" "Not in stock"
+			(at 69.85 130.81 0)
+			(effects
+				(font
+					(size 1.27 1.27)
+				)
+				(justify bottom)
+				(hide yes)
+			)
+		)
+		(property "MANUFACTURER" "Espressif"
+			(at 69.85 130.81 0)
+			(effects
+				(font
+					(size 1.27 1.27)
+				)
+				(justify bottom)
+				(hide yes)
+			)
+		)
+		(pin "1"
+		)
+		(pin "2"
+		)
+		(pin "0"
+		)
+		(pin "3"
+		)
+		(pin "8"
+		)
+		(pin "9"
+		)
+		(pin "G"
+		)
+		(pin "21"
+		)
+		(pin "3.3"
+		)
+		(pin "20"
+		)
+		(pin "6"
+		)
+		(pin "5"
+		)
+		(pin "4"
+		)
+		(pin "7"
+		)
+		(pin "5V"
+		)
+		(pin "10"
+		)
+		(instances
+			(project ""
+				(path "/50c2c19d-4e9f-46ca-96ff-b8e974e917a5"
+					(reference "U4")
+					(unit 1)
+				)
+			)
+		)
 	)
 	(symbol

Commit message: Aku VCU
Connections:
- net GND: now also J1.14 (Pin_14), J1.15 (Pin_15), J1.16 (Pin_16), J1.4 (Pin_4), J1.5 (Pin_5), J2.6 (Pin_6), J2.7 (Pin_7), J2.8 (Pin_8), J2.9 (Pin_9)
