File: Bimasakti BM-13 EVO/PCB/VCU/_autosave-VCU.kicad_pcb (KiCad board)
At the start: 2 copper layers, 84 x 88.5 mm, 79 parts, among them J1 Conn_01x28_Pin, J2 Conn_01x28_Pin, K1 IM00, K2 IM00, K3 IM00, Q1 SQ2362CES, Q2 SQ2362CES, Q3 SQ2362CES, Q4 DMTH6004SK3, Q5 DMTH6004SK3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

Commit message: Aku VCU
Parts:
- added G***: LOGO, Bimsak:aaaaaaaa, F.Cu at (110.1, 149.9)
Other:
- board text added: "- VCU (Vehicle Control Unit)-"
- board text added: "BM - 13 Hybrid"
