File: Bimasakti BM-13 EVO/PCB/VCU/VCU.kicad_pcb (KiCad board)
At the start: 2 copper layers, 70 parts, among them J1 Conn_01x26_Pin, J2 Conn_01x26_Pin, K1 IM00, K2 IM00, K3 IM00, Q1 SQ2362CES, Q2 SQ2362CES, Q3 SQ2362CES, Q4 DMTH6004SK3, Q5 DMTH6004SK3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

Commit message: Aku VCU
Parts:
- added D13: LED, LED_SMD:LED_0603_1608Metric_Pad1.05x0.95mm_HandSolder, F.Cu at (131.4, 79.2)
- added R31: 1K, Resistor_SMD:R_0603_1608Metric_Pad0.98x0.95mm_HandSolder, F.Cu at (135.2, 79.2)
- added R32: R_Small_US, Resistor_SMD:R_0603_1608Metric_Pad0.98x0.95mm_HandSolder, F.Cu at (138.1, 94.1)
- added R33: R_Small_US, Resistor_SMD:R_0603_1608Metric_Pad0.98x0.95mm_HandSolder, F.Cu at (138.2, 84.2)
- added R34: R_Small_US, Resistor_SMD:R_0603_1608Metric_Pad0.98x0.95mm_HandSolder, F.Cu at (138.2, 103.6)
- added REF**: MountingHole_3.2mm_M3_Pad_Via, MountingHole:MountingHole_3.2mm_M3_Pad_Via, F.Cu at (149.0, 73.0)
- added REF**: MountingHole_3.2mm_M3_Pad_Via, MountingHole:MountingHole_3.2mm_M3_Pad_Via, F.Cu at (75.0, 73.0)
- added REF**: MountingHole_3.2mm_M3_Pad_Via, MountingHole:MountingHole_3.2mm_M3_Pad_Via, F.Cu at (149.0, 151.5)
- added REF**: MountingHole_3.2mm_M3_Pad_Via, MountingHole:MountingHole_3.2mm_M3_Pad_Via, F.Cu at (75.0, 151.5)
- J1, J2: value Conn_01x26_Pin -> Conn_01x28_Pin; footprint Connector_PinHeader_2.54mm:PinHeader_1x26_P2.54mm_Vertical -> Connector_PinHeader_2.54mm:PinHeader_1x28_P2.54mm_Vertical
- moved R19 48.3 mm to (103.0, 131.0)
- moved R23 46.1 mm to (97.1, 131.0), turned to -90 degrees
- moved D10 45.4 mm to (100.0, 130.1)
- moved U6 45.2 mm to (100.3, 134.8)
- moved R27 44.3 mm to (100.0, 131.9), turned to 180 degrees
- moved Q4 43.8 mm to (89.0, 133.1), turned to 180 degrees
- moved D5 38.9 mm to (100.3, 137.3), turned to 180 degrees
- moved R21 35.0 mm to (103.2, 120.4)
- moved R25 32.5 mm to (97.4, 120.5), turned to -90 degrees
- moved Q5 31.4 mm to (89.0, 122.7), turned to 180 degrees
- moved U8 28.2 mm to (100.4, 124.1)
- moved R20 26.9 mm to (103.2, 141.6)
- moved D11 26.8 mm to (100.2, 119.5)
- moved R29 25.8 mm to (100.2, 121.3), turned to 180 degrees
- moved D6 25.1 mm to (100.3, 126.7), turned to 180 degrees
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Connections:
- BMS1 pad 8: unconnected-(BMS1-RS-Pad8) -> Net-(BMS1-RS)
- D5 pad 2: +5V -> +5VA
- D6 pad 2: +5V -> +5VA
- D7 pad 2: +5V -> +5VA
- D8 pad 2: +5V -> +5VA
- Display1 pad 8: unconnected-(Display1-RS-Pad8) -> Net-(Display1-RS)
- ECU1 pad 8: unconnected-(ECU1-RS-Pad8) -> Net-(ECU1-RS)
- J1 pad 10: unconnected-(J1-Pin_10-Pad10) -> /SDC_OUT
- J1 pad 11: unconnected-(J1-Pin_11-Pad11) -> /Brake_Light
- J1 pad 12: unconnected-(J1-Pin_12-Pad12) -> /FAN_BATT
- J1 pad 13: unconnected-(J1-Pin_13-Pad13) -> GND
- J1 pad 14: unconnected-(J1-Pin_14-Pad14) -> /TX_TV
- J1 pad 15: unconnected-(J1-Pin_15-Pad15) -> GND
- J1 pad 16: unconnected-(J1-Pin_16-Pad16) -> /RX_TV
- J1 pad 17: /Safety -> GND
- J1 pad 18: /Engine -> GND
- J1 pad 19: /PDM -> /CS_T
- J1 pad 20: /AIR -> GND
- J1 pad 21: /Hybrid -> /MOSI_T
- J1 pad 22: /FAN_BATT -> GND
- J1 pad 23: /Brake_Light -> /MISO_T
- J1 pad 24: /SWITCH -> GND
- J1 pad 25: /SDC_IN -> /SCK_T
- J1 pad 26: /SDC_OUT -> GND
- J1 pad 3: /CS_T -> /Engine
- J1 pad 4: /MOSI_T -> /PDM
- J1 pad 5: /MISO_T -> /Safety
- J1 pad 6: /SCK_T -> /Hybrid
- J1 pad 7: GND -> /AIR
- J1 pad 8: unconnected-(J1-Pin_8-Pad8) -> /Safety
- J1 pad 9: unconnected-(J1-Pin_9-Pad9) -> /SDC_IN
- J2 pad 10: /Ac3 -> /CANH_3
- J2 pad 11: /Ac4 -> /CANL_3
- J2 pad 16: /CANH_1 -> /Ac4
- J2 pad 17: /CANL_1 -> /Ac3
- J2 pad 18: GND -> /Ac2
- J2 pad 19: /CANH_2 -> /Brake_Pressure
- J2 pad 2: /Analog1 -> GND
- J2 pad 20: /CANL_2 -> GND
- J2 pad 21: GND -> /SUS4
- J2 pad 22: /CANH_3 -> /SUS3
- J2 pad 23: /CANL_3 -> /SUS2
- J2 pad 24: GND -> /SUS1
- J2 pad 26: GND -> /Analog2
- J2 pad 3: /Analog2 -> GND
- J2 pad 4: /SUS1 -> /CANH_2
- J2 pad 5: /SUS2 -> /CANL_2
- J2 pad 6: /SUS3 -> GND
- J2 pad 7: /SUS4 -> /CANH_1
- J2 pad 8: /Brake_Pressure -> /CANL_1
- J2 pad 9: /Ac2 -> GND
- K1 pad 6: +3.3V -> +3.3VA
- K2 pad 6: +3.3V -> +3.3VA
- Teensy4.1 pad 11: /D1_BATT -> /D3
- Teensy4.1 pad 15: +3.3V -> +3.3VA
- Teensy4.1 pad 46: +3.3VA -> +3.3V
- Teensy4.1 pad 7: /D3 -> /D2_BL
- Teensy4.1 pad 8: /D2_BL -> /D1_BATT
- U6 pad 4: +5V -> +5VA
- U7 pad 4: +5V -> +5VA
- U8 pad 4: +5V -> +5VA
- U9 pad 4: +5V -> +5VA
Routing:
- net +12V: track 22.6 -> 218.8 mm, vias 0 -> 5
- net +3.3V: track 0.00 -> 148.4 mm, vias 0 -> 5
- net +3.3VA: track 0.00 -> 84.0 mm
- net +5VA: track 0.00 -> 72.5 mm, vias 0 -> 4
- net /SCK_T: track 0.00 -> 70.5 mm
- net /CRX3: track 0.00 -> 67.1 mm
- net /CTX3: track 0.00 -> 66.4 mm
- net +5V: track 0.11 -> 65.1 mm, vias 0 -> 4
- net /Analog1: track 0.00 -> 50.9 mm
- net /FAN_BATT: track 0.00 -> 47.3 mm
- net /Analog2: track 0.00 -> 44.9 mm
- net /SDA: track 0.00 -> 43.3 mm, vias 0 -> 1
- net /SCL: track 0.00 -> 42.1 mm, vias 0 -> 2
- net /Brake_Light: track 0.00 -> 40.6 mm
- net /CTX2: track 0.00 -> 39.0 mm
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- added copper zone on B.Cu, net GND
- added copper zone on F.Cu, net GND
Other:
- board outline added: 84 x 88.5 mm
- board text added: "Analog_ _16_Bit"
- board text added: "BMS"
- board text added: "Brake_Light"
- board text added: "Display"
- board text added: "ECU"
- board text added: "ENGINE"
- board text added: "FAN_Batt"
- board text added: "HYBRID"
- board text added: "SAFETY"
- board text added: "Switch"

Commit message: VCU Finish
Parts:
- added G***: LOGO, Bimsak:aaaaaaaa, F.Cu at (110.9, 149.3)
- added REF**: ESD-Logo_6.6x6mm_SilkScreen, Symbol:ESD-Logo_6.6x6mm_SilkScreen, B.Cu at (135.8, 149.6)
Other:
- board text added: "- VCU (Vehicle Control Unit)-"
- board text added: "BM - 13 Hybrid"
- board text added: "Feature VCU - Teensy 4.1 - 8 Pin Analog 16 Bit - 2 Pin Analog 10 Bit - 3 CAN Bus - 3 Switch High Side - 3 Switch Low Side - 1 UART - 1 SPI"
- board text added: "PCB Ini dibuat dengan Kopi dan Malboro Kretek Dalam waktu 1 Minggu di Kesindirian yang sunyi"

Commit message: Aku Pneumatic
Connections:
- J2 pad 14: GND -> /Ac4
- J2 pad 15: GND -> /Ac3
- J2 pad 16: /Ac4 -> /Ac2
- J2 pad 17: /Ac3 -> /Brake_Pressure
- J2 pad 18: /Ac2 -> /SUS4
- J2 pad 19: /Brake_Pressure -> /SUS3
- J2 pad 20: GND -> /SUS2
- J2 pad 21: /SUS4 -> /SUS1
- J2 pad 22: /SUS3 -> GND
- J2 pad 23: /SUS2 -> /RX_Pneu
- J2 pad 24: /SUS1 -> /TX_Pneu
- Teensy4.1 pad 26: unconnected-(Teensy4.1-RX8-Pad26) -> /TX_Pneu
- Teensy4.1 pad 27: unconnected-(Teensy4.1-TX8-Pad27) -> /RX_Pneu
Routing:
- net /RX_Pneu: track 0.00 -> 26.8 mm
- net /TX_Pneu: track 0.00 -> 24.9 mm
- net /SUS4: track 7.70 -> 14.3 mm
- net /SUS3: track 6.82 -> 13.3 mm
- net /Ac4: track 7.86 -> 11.5 mm
- net /Ac3: track 7.01 -> 10.5 mm
- net /SUS2: track 7.53 -> 10.8 mm
- net /Brake_Pressure: track 8.97 -> 7.43 mm
- net /Analog1: track 50.9 -> 50.3 mm
- net GND: track 38.3 -> 38.5 mm, vias 269 -> 296
