File: Bimasakti BM-13 EVO/PCB/VCU/VCU.kicad_pcb (KiCad board)
At the start: 2 copper layers, 84 x 88.5 mm, 76 parts, among them J1 Conn_01x28_Pin, J2 Conn_01x28_Pin, K1 IM00, K2 IM00, K3 IM00, Q1 SQ2362CES, Q2 SQ2362CES, Q3 SQ2362CES, Q4 DMTH6004SK3, Q5 DMTH6004SK3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

Commit message: tambah i2c di tele
Connections:
- J2 pad 2: GND -> /SDA
- J2 pad 3: GND -> /SCL
- U1 pad 10: /SUS4 -> SUSP4
- U1 pad 7: /SUS1 -> SUSP1
- U1 pad 8: /SUS2 -> SUSP2
- U1 pad 9: /SUS3 -> SUSP3
- U2 pad 10: /Ac4 -> A4
- U2 pad 7: /Brake_Pressure -> BRK_P
- U2 pad 8: /Ac2 -> A2
- U2 pad 9: /Ac3 -> A3
Routing:
- net /SDA: track 42.9 -> 101.9 mm
- net /SCL: track 42.1 -> 94.8 mm
- net SUSP4: track 0.00 -> 14.3 mm
- net /SUS4: track 14.3 -> 0.00 mm
- net SUSP3: track 0.00 -> 13.5 mm
- net /SUS3: track 13.3 -> 0.00 mm
- net A4: track 0.00 -> 12.5 mm
- net /TX_TV: track 68.7 -> 57.2 mm
- net /Ac4: track 11.5 -> 0.00 mm
- net SUSP2: track 0.00 -> 10.8 mm
- net /SUS2: track 10.8 -> 0.00 mm
- net A3: track 0.00 -> 10.5 mm
- net /Ac3: track 10.5 -> 0.00 mm
- net SUSP1: track 0.00 -> 8.82 mm
- net /SUS1: track 8.82 -> 0.00 mm
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