File: Bimasakti BM-13 EVO/PCB/VCU/VCU.kicad_sch (KiCad schematic)
At the start: 0 parts

Commit message: Aku VCU
Parts:
- added BMS1, Display1, ECU1: SN65HVD230D, SN65HVD230D:SOIC127P599X175-8N, symbol SN65HVD230D:SN65HVD230D
- added C1, C2, C3, C4, C5: 100nF, symbol Device:C_Small
- added J1, J2: Conn_01x03_Pin, symbol Connector:Conn_01x03_Pin
- added Q1, Q2, Q3, Q4, Q5: BS107, Package_TO_SOT_THT:TO-92_Inline, symbol Transistor_FET:BS107
- added R1, R3, R5: 120, symbol Device:R_Small_US
- added R10, R7, R8, R9: 4.7K, symbol Device:R_Small_US
- added R2, R4, R6: 0, symbol Device:R_Small_US
- added Teensy4.1: ~, teensy:Teensy41, symbol teensy41:teensy4.1
- added U1, U2: ~, Custom_ADS:ADS1115, symbol ads1115:ADS1115
- added U3, U4, U5: 6N137, Package_DIP:DIP-8_W7.62mm, symbol Isolator:6N137
Connections:
- new net: BMS1.5 (VREF), R2.1
- new net: BMS1.6 (CANL), R1.2
- new net: BMS1.7 (CANH), R1.1
- new net: ECU1.7 (CANH), R3.1
- new net: ECU1.6 (CANL), R3.2
- new net: Display1.5 (VREF), R6.1
- new net: Display1.6 (CANL), R5.2
- new net: Display1.7 (CANH), R5.1
- new net: ECU1.5 (VREF), R4.1
- new net +3.3V: BMS1.3 (VCC), C1.2, C2.2, C3.2, C4.2, C5.2, Display1.3 (VCC), ECU1.3 (VCC), J1.1 (Pin_1), J2.1 (Pin_1), R10.2, R7.2, R8.2, R9.2, U1.1 (VDD), U2.1 (VDD)
- new net ADR1: J1.2 (Pin_2), U1.5 (ADDR)
- new net ADR2: J2.2 (Pin_2), U2.5 (ADDR)
- new net Ac1: U2.7 (A0)
- new net Ac2: U2.8 (A1)
- new net Ac3: U2.9 (A2)
- new net Ac4: U2.10 (A3)
- new net CRX1: BMS1.4 (R)
- new net CRX2: ECU1.4 (R)
- new net CRX3: Display1.4 (R)
- new net CTX1: BMS1.1 (D)
- new net CTX2: ECU1.1 (D)
- new net CTX3: Display1.1 (D)
- new net GND: BMS1.2 (GND), C1.1, C2.1, C3.1, C4.1, C5.1, Display1.2 (GND), ECU1.2 (GND), J1.3 (Pin_3), J2.3 (Pin_3), R2.2, R4.2, R6.2, U1.2 (GND), U2.2 (GND)
- new net SCL: R10.1, R8.1, U1.3 (SCL), U2.3 (SCL)
- new net SDA: R7.1, R9.1, U1.4 (SDA), U2.4 (SDA)
- new net SUS1: U1.7 (A0)
- new net SUS2: U1.8 (A1)
- new net SUS3: U1.9 (A2)
- new net SUS4: U1.10 (A3)

Commit message: Aku VCU
Parts:
- removed Q1, Q2, Q3, Q4, Q5: BS107, Package_TO_SOT_THT:TO-92_Inline, symbol Transistor_FET:BS107
- removed U3, U4, U5: 6N137, Package_DIP:DIP-8_W7.62mm, symbol Isolator:6N137
- added D1, D2, D5, D6, D7, D8: LED, symbol Device:LED
- added D3, D4, D9: D, symbol Device:D
- added J1, J2: Conn_01x26_Pin, symbol Connector:Conn_01x26_Pin
- added K1, K2, K3: IM00, Relay TE Small 5 Amp:RELAY8-TH_NON-LATCH_1-COIL, symbol Relay:IM00
- added Q11, Q12, Q13, Q14: IPD040N03LF2S, Package_TO_SOT_THT:TO-18-3, symbol Transistor_BJT:BC107
- added Q6, Q7: SQ2318AES, Package_TO_SOT_THT:TO-18-3, symbol Transistor_BJT:BC107
- added R11, R12, R13, R15, R27, R28, R29, R30: 1K, symbol Device:R_Small_US
- added R14, R16, R17, R18, R23, R24, R25, R26: 10K, symbol Device:R_Small_US
- added R19, R20, R21, R22: 330, symbol Device:R_Small_US
- added U6, U7, U8, U9: TCMT1103, Package_SO:SOP-4_4.4x2.6mm_P1.27mm, symbol Isolator:TCMT1103
- BMS1, Display1, ECU1: footprint SN65HVD230D:SOIC127P599X175-8N -> CAN Tranciver:SOIC127P599X175-8N
- renumbered J1 to ADS1, J2 to ADS2
Connections:
- net +3.3V: now also K1.6, K2.6
- net Ac2: now also J1.8 (Pin_8)
- net Ac3: now also J1.9 (Pin_9)
- net Ac4: now also J1.10 (Pin_10)
- net CRX1: now also Teensy4.1.45 (A9/CRX1)
- net CRX2: now also Teensy4.1.2 (RX1)
- net CRX3: now also Teensy4.1.22 (CRX3)
- net CTX1: now also Teensy4.1.44 (A8/CTX1)
- net CTX2: now also Teensy4.1.3 (TX1)
- net CTX3: now also Teensy4.1.23 (CTX3)
- net GND: now also Teensy4.1.1 (GND), J2.11 (Pin_11), J2.2 (Pin_2), J2.5 (Pin_5), J2.8 (Pin_8), K3.5, Q11.1 (E), Q12.1 (E), Q13.1 (E), Q14.1 (E), Q6.1 (E), Q7.1 (E), R14.2, R16.2, R17.2, R18.2, R23.1, R24.1, R25.1, R26.1, U6.2, U7.2, U8.2, U9.2
- net SCL: now also Teensy4.1.41 (A5/SCL)
- net SDA: now also Teensy4.1.40 (A4/SDA)
- net SUS1: now also J1.3 (Pin_3)
- net SUS2: now also J1.4 (Pin_4)
- net SUS3: now also J1.5 (Pin_5)
- net SUS4: now also J1.6 (Pin_6)
- net RX_TV: now reaches Teensy4.1.10 (IN1)
- net D4_SDC: now reaches Teensy4.1.11 (OUT1C)
- net D4_SDC: now also R22.1
- net CS_T: now reaches Teensy4.1.12 (MQSR)
- net CS_T: now also J1.13 (Pin_13)
- net MOSI_T: now reaches Teensy4.1.13 (CTX1)
- net MOSI_T: now also J1.14 (Pin_14)
- net MISO_T: now reaches Teensy4.1.14 (MQSL)
- net MISO_T: now also J1.15 (Pin_15)
- net SCK_T: now reaches Teensy4.1.35 (SCK/LED)
- net SCK_T: now also J2.15 (Pin_15)
- net IND_Hybrid: now reaches Teensy4.1.4 (OUT2)
- net IND_Hybrid: now also K2.7, R17.1
- net +5V: now reaches Teensy4.1.48 (Vin)
- net +5V: now also D5.2 (A), D6.2 (A), D7.2 (A), D8.2 (A), J2.1 (Pin_1), R11.1, R12.1
- net IND_Engine: now reaches Teensy4.1.5 (LRCLK2)
- net IND_Engine: now also K1.7, R18.1
- net D1_BATT: now reaches Teensy4.1.6 (BCLK2)
- net D1_BATT: now also R19.1
- net D2_BL: now reaches Teensy4.1.7 (IN2)
- net D2_BL: now also R21.1
- net D3: now reaches Teensy4.1.8 (OUT1D)
- net D3: now also R20.1
- net TX_TV: now reaches Teensy4.1.9 (OUT1A)
- net CANL_1: now reaches BMS1.6 (CANL), R1.2
- net CANL_1: now also J2.4 (Pin_4)
- net CANH_1: now reaches BMS1.7 (CANH), R1.1
- net CANH_1: now also J2.3 (Pin_3)
- net CANH_2: now reaches ECU1.7 (CANH), R3.1
- net CANH_2: now also J2.6 (Pin_6)
- net CANL_2: now reaches ECU1.6 (CANL), R3.2
- net CANL_2: now also J2.7 (Pin_7)
- net CANL_3: now reaches Display1.6 (CANL), R5.2
- net CANL_3: now also J2.10 (Pin_10)
- net CANH_3: now reaches Display1.7 (CANH), R5.1
- net CANH_3: now also J2.9 (Pin_9)
- net Ac1 renamed Brake_Pressure
- net Brake_Pressure: now also J1.7 (Pin_7)
- new net: D2.2 (A), R12.2
- new net: Q13.2 (B), R26.2, U9.3
- new net: D9.2 (A), K3.8, Q13.3 (C)
- new net: D1.1 (K), D3.2 (A), K1.8, Q6.3 (C)
- new net: R20.2, U7.1
- new net: Q6.2 (B), R13.2, R14.1
- new net: D7.1 (K), R28.1
- new net: R28.2, U7.4
- new net: D2.1 (K), D4.2 (A), K2.8, Q7.3 (C)
- new net: Q7.2 (B), R15.2, R16.1
- new net: D8.1 (K), R30.1
- new net: R30.2, U9.4
- new net: D5.1 (K), R27.1
- new net: Q12.2 (B), R25.2, U8.3
- new net: D6.1 (K), R29.1
- new net: R29.2, U8.4
- new net: Q14.2 (B), R23.2, U6.3
- new net: R22.2, U9.1
- new net: R21.2, U8.1
- new net: D1.2 (A), R11.2
- new net: R19.2, U6.1
- new net: Q11.2 (B), R24.2, U7.3
- new net: R27.2, U6.4
- new net +12V: D3.1 (K), D4.1 (K), D9.1 (K), J1.1 (Pin_1), K1.1, K2.1, K3.1
- new net AIR: K2.2
- new net Brake_Light: Q12.3 (C)
- new net Engine: J1.20 (Pin_20), R13.1
- new net FAN_BATT: Q14.3 (C)
- new net Hybrid: J1.18 (Pin_18), R15.1
- new net LED_SDC: K3.6
- new net PDM: K1.2
- new net SDC_IN: K3.3
- new net SDC_OUT: K3.4
- new net SWITCH: Q11.3 (C)
- new net Safety: J1.19 (Pin_19), K1.3, K2.3
Other:
- note added: "ADS"
- note added: "Address ADS1"
- note added: "Address ADS2"
- note added: "BMS"
- note added: "CAN Tranciver"
- note added: "Display"
- note added: "ECU"
- note added: "Safety Engine"
- note added: "Safety Hybrid"
- moved on the sheet: ADS1, ADS2, BMS1, C1, C2, C3, C4, C5, Display1, ECU1, R1, R10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

Commit message: Aku VCU
Parts:
- removed Q11, Q12, Q13, Q14: IPD040N03LF2S, Package_TO_SOT_THT:TO-18-3, symbol Transistor_BJT:BC107
- removed Q6, Q7: SQ2318AES, Package_TO_SOT_THT:TO-18-3, symbol Transistor_BJT:BC107
- added D10, D11, D12: D, Diode_SMD:D_0603_1608Metric_Pad1.05x0.95mm_HandSolder, symbol Device:D
- added Q1, Q2, Q3: SQ2362CES, Package_TO_SOT_SMD:SOT-23, symbol Transistor_FET:2N7002K
- added Q4, Q5, Q6: DMTH6004SK3, Package_TO_SOT_SMD:TO-252-2, symbol Transistor_FET:BSP89
- ADS1, ADS2: footprint (none) -> Connector_PinHeader_2.54mm:PinHeader_1x03_P2.54mm_Vertical
- C1, C2, C3, C4, C5: footprint (none) -> Capacitor_SMD:C_0603_1608Metric_Pad1.08x0.95mm_HandSolder
- D1, D2, D5, D6, D7, D8: footprint (none) -> LED_SMD:LED_0603_1608Metric_Pad1.05x0.95mm_HandSolder
- D3, D4, D9: footprint (none) -> Diode_SMD:D_0603_1608Metric_Pad1.05x0.95mm_HandSolder
- J1, J2: footprint (none) -> Connector_PinHeader_2.54mm:PinHeader_1x26_P2.54mm_Vertical
- R1, R10, R13, R14, R15, R16, R17, R18, R19, R2, R20, R21, R22, R23, R24, R25, R26, R27, R28, R29, R3, R30, R4, R5, R6, R7, R8, R9: footprint (none) -> Resistor_SMD:R_0603_1608Metric_Pad0.98x0.95mm_HandSolder
- R11, R12: value 1K -> 330; footprint (none) -> Resistor_SMD:R_0603_1608Metric_Pad0.98x0.95mm_HandSolder
- U1, U2: footprint Custom_ADS:ADS1115 -> ADS1115:MSOP10
Connections:
- net +12V: now also D10.1 (K), D11.1 (K), D12.1 (K)
- net +3.3V: now also Teensy4.1.15 (3.3V)
- net +5V: now also U6.4, U7.4, U8.4, U9.4
- net AIR: now also J1.20 (Pin_20)
- net Ac2: now also J2.9 (Pin_9); no longer J1.8 (Pin_8)
- net Ac3: now also J2.10 (Pin_10); no longer J1.9 (Pin_9)
- net Ac4: now also J2.11 (Pin_11); no longer J1.10 (Pin_10)
- net Brake_Light: now also J1.23 (Pin_23), R29.2, D11.2 (A), Q5.2 (D)
- net Brake_Pressure: now also J2.8 (Pin_8); no longer J1.7 (Pin_7)
- net CANH_1: now also J2.16 (Pin_16); no longer J2.3 (Pin_3)
- net CANH_2: now also J2.19 (Pin_19); no longer J2.6 (Pin_6)
- net CANH_3: now also J2.22 (Pin_22); no longer J2.9 (Pin_9)
- net CANL_1: now also J2.17 (Pin_17); no longer J2.4 (Pin_4)
- net CANL_2: now also J2.20 (Pin_20); no longer J2.7 (Pin_7)
- net CANL_3: now also J2.23 (Pin_23); no longer J2.10 (Pin_10)
- net CS_T: now also J1.3 (Pin_3); no longer J1.13 (Pin_13)
- net D1_BATT: now also Teensy4.1.11 (OUT1C); no longer Teensy4.1.6 (BCLK2)
- net D2_BL: now also Teensy4.1.8 (OUT1D); no longer Teensy4.1.7 (IN2)
- net D3: now also Teensy4.1.7 (IN2); no longer Teensy4.1.8 (OUT1D)
- net D4_SDC: now also Teensy4.1.6 (BCLK2); no longer Teensy4.1.11 (OUT1C)
- net Engine: now also J1.18 (Pin_18); no longer J1.20 (Pin_20)
- net FAN_BATT: now also J1.22 (Pin_22), R27.2, D10.2 (A), Q4.2 (D)
- net GND: now also J1.2 (Pin_2), J1.7 (Pin_7), J2.12 (Pin_12), J2.13 (Pin_13), J2.14 (Pin_14), J2.15 (Pin_15), J2.18 (Pin_18), J2.21 (Pin_21), J2.24 (Pin_24), J2.25 (Pin_25), J2.26 (Pin_26), K3.7, Teensy4.1.34 (GND), Teensy4.1.47 (GND), Q1.2 (S), Q2.2 (S), Q3.2 (S), Q4.3 (S), Q5.3 (S), Q6.3 (S); no longer J2.11 (Pin_11), J2.2 (Pin_2), J2.5 (Pin_5), J2.8 (Pin_8), K3.5
- net Hybrid: now also J1.21 (Pin_21); no longer J1.18 (Pin_18)
- net IND_Engine: now also R17.1, Teensy4.1.4 (OUT2); no longer R18.1, Teensy4.1.5 (LRCLK2)
- net IND_Hybrid: now also R18.1, Teensy4.1.5 (LRCLK2); no longer R17.1, Teensy4.1.4 (OUT2)
- net LED_SDC: now also R30.2
- net MISO_T: now also J1.5 (Pin_5); no longer J1.15 (Pin_15)
- net MOSI_T: now also J1.4 (Pin_4); no longer J1.14 (Pin_14)
- net PDM: now also J1.19 (Pin_19)
- net SCK_T: now also J1.6 (Pin_6); no longer J2.15 (Pin_15)
- net SDC_IN: now also J1.25 (Pin_25)
- net SDC_OUT: now also J1.26 (Pin_26)
- net SUS1: now also J2.4 (Pin_4); no longer J1.3 (Pin_3)
- net SUS2: now also J2.5 (Pin_5); no longer J1.4 (Pin_4)
- net SUS3: now also J2.6 (Pin_6); no longer J1.5 (Pin_5)
- net SUS4: now also J2.7 (Pin_7); no longer J1.6 (Pin_6)
- net SWITCH: now also J1.24 (Pin_24), R28.2, D12.2 (A), Q6.2 (D)
- net Safety: now also J1.17 (Pin_17); no longer J1.19 (Pin_19)
- net Analog2: now reaches Teensy4.1.32 (A16)
- net Analog2: now also J2.3 (Pin_3)
- net Analog1: now reaches Teensy4.1.33 (A17)
- net Analog1: now also J2.2 (Pin_2)
- net +3.3VA: now reaches Teensy4.1.46 (3.3V)
- net at R26.2, U9.3: now also Q3.1 (G)
- net at D9.2 (A), K3.8: now also Q3.3 (D)
- net at D1.1 (K), D3.2 (A), K1.8: now also Q1.3 (D)
- net at R13.2, R14.1: now also Q1.1 (G)
- net at D2.1 (K), D4.2 (A), K2.8: now also Q2.3 (D)
- net at R15.2, R16.1: now also Q2.1 (G)
- net at R25.2, U8.3: now also Q5.1 (G)
- net at R23.2, U6.3: now also Q4.1 (G)
- net at R24.2, U7.3: now also Q6.1 (G)
Other:
- note added: "Brake Light"
- note added: "FAN Battery"
- note added: "SDC Hybrid_Control"
- note added: "Switch"
- moved on the sheet: ADS1, ADS2, C4, C5, D1, D2, D3, D4, D5, D6, D7, D8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

Commit message: Aku VCU
Parts:
- removed J1, J2: Conn_01x26_Pin, Connector_PinHeader_2.54mm:PinHeader_1x26_P2.54mm_Vertical, symbol Connector:Conn_01x26_Pin
- added D13: LED, LED_SMD:LED_0603_1608Metric_Pad1.05x0.95mm_HandSolder, symbol Device:LED
- added J1, J2: Conn_01x28_Pin, Connector_PinHeader_2.54mm:PinHeader_1x28_P2.54mm_Vertical, symbol Connector:Conn_01x28_Pin
- added R31: 1K, Resistor_SMD:R_0603_1608Metric_Pad0.98x0.95mm_HandSolder, symbol Device:R_Small_US
- added R32, R33, R34: R_Small_US, Resistor_SMD:R_0603_1608Metric_Pad0.98x0.95mm_HandSolder, symbol Device:R_Small_US
Connections:
- net +12V: now also J1.1 (Pin_1)
- net +3.3V: now also Teensy4.1.46 (3.3V); no longer K1.6, K2.6, Teensy4.1.15 (3.3V)
- net +3.3VA: now also K1.6, K2.6, Teensy4.1.15 (3.3V); no longer Teensy4.1.46 (3.3V)
- net +5V: now also J2.1 (Pin_1), R31.1; no longer D5.2 (A), D6.2 (A), D7.2 (A), D8.2 (A), U6.4, U7.4, U8.4, U9.4
- net AIR: now also J1.7 (Pin_7)
- net Ac2: now also J2.18 (Pin_18)
- net Ac3: now also J2.17 (Pin_17)
- net Ac4: now also J2.16 (Pin_16)
- net Analog1: now also J2.27 (Pin_27)
- net Analog2: now also J2.26 (Pin_26)
- net Brake_Light: now also J1.11 (Pin_11)
- net Brake_Pressure: now also J2.19 (Pin_19)
- net CANH_1: now also J2.7 (Pin_7)
- net CANH_2: now also J2.4 (Pin_4)
- net CANH_3: now also J2.10 (Pin_10)
- net CANL_1: now also J2.8 (Pin_8)
- net CANL_2: now also J2.5 (Pin_5)
- net CANL_3: now also J2.11 (Pin_11)
- net CS_T: now also J1.19 (Pin_19)
- net D1_BATT: now also Teensy4.1.8 (OUT1D); no longer Teensy4.1.11 (OUT1C)
- net D2_BL: now also Teensy4.1.7 (IN2); no longer Teensy4.1.8 (OUT1D)
- net D3: now also Teensy4.1.11 (OUT1C); no longer Teensy4.1.7 (IN2)
- net Engine: now also J1.3 (Pin_3)
- net FAN_BATT: now also J1.12 (Pin_12)
- net GND: now also D13.1 (K), J1.13 (Pin_13), J1.15 (Pin_15), J1.17 (Pin_17), J1.18 (Pin_18), J1.2 (Pin_2), J1.20 (Pin_20), J1.22 (Pin_22), J1.24 (Pin_24), J1.26 (Pin_26), J2.12 (Pin_12), J2.13 (Pin_13), J2.14 (Pin_14), J2.15 (Pin_15), J2.2 (Pin_2), J2.20 (Pin_20), J2.25 (Pin_25), J2.28 (Pin_28), J2.3 (Pin_3), J2.6 (Pin_6), J2.9 (Pin_9), R32.2, R33.2, R34.2
- net Hybrid: now also J1.6 (Pin_6)
- net MISO_T: now also J1.23 (Pin_23)
- net MOSI_T: now also J1.21 (Pin_21)
- net PDM: now also J1.4 (Pin_4)
- net RX_TV: now also J1.16 (Pin_16)
- net SCK_T: now also J1.25 (Pin_25)
- net SDC_IN: now also J1.9 (Pin_9)
- net SDC_OUT: now also J1.10 (Pin_10)
- net SUS1: now also J2.24 (Pin_24)
- net SUS2: now also J2.23 (Pin_23)
- net SUS3: now also J2.22 (Pin_22)
- net SUS4: now also J2.21 (Pin_21)
- net SWITCH: now also J1.27 (Pin_27)
- net Safety: now also J1.5 (Pin_5), J1.8 (Pin_8)
- net TX_TV: now also J1.14 (Pin_14)
- net at BMS1.8 (RS): now also R32.1
- net at Display1.8 (RS): now also R34.1
- net at ECU1.8 (RS): now also R33.1
- new net: D13.2 (A), R31.2
- new net +5VA: D5.2 (A), D6.2 (A), D7.2 (A), D8.2 (A), J1.28 (Pin_28), U6.4, U7.4, U8.4, U9.4

Commit message: Aku Pneumatic
Connections:
- net Ac2: now also J2.16 (Pin_16); no longer J2.18 (Pin_18)
- net Ac3: now also J2.15 (Pin_15); no longer J2.17 (Pin_17)
- net Ac4: now also J2.14 (Pin_14); no longer J2.16 (Pin_16)
- net Brake_Pressure: now also J2.17 (Pin_17); no longer J2.19 (Pin_19)
- net GND: now also J2.22 (Pin_22); no longer J2.14 (Pin_14), J2.15 (Pin_15), J2.20 (Pin_20)
- net SUS1: now also J2.21 (Pin_21); no longer J2.24 (Pin_24)
- net SUS2: now also J2.20 (Pin_20); no longer J2.23 (Pin_23)
- net SUS3: now also J2.19 (Pin_19); no longer J2.22 (Pin_22)
- net SUS4: now also J2.18 (Pin_18); no longer J2.21 (Pin_21)
- net TX_Pneu: now reaches Teensy4.1.26 (RX8)
- net TX_Pneu: now also J2.24 (Pin_24)
- net RX_Pneu: now reaches Teensy4.1.27 (TX8)
- net RX_Pneu: now also J2.23 (Pin_23)

Commit message: Asu
Parts:
- added R35, R36, R37, R38, R39, R45, R47, R49: 2K, Resistor_SMD:R_0402_1005Metric_Pad0.72x0.64mm_HandSolder, symbol Device:R
- added R40, R41, R42, R43, R44, R46, R48, R50: 3K, Resistor_SMD:R_0402_1005Metric_Pad0.72x0.64mm_HandSolder, symbol Device:R
Connections:
- net Ac2: now also R45.1, R46.1; no longer J2.16 (Pin_16)
- net Ac3: now also R47.1, R48.1; no longer J2.15 (Pin_15)
- net Ac4: now also R49.1, R50.1; no longer J2.14 (Pin_14)
- net Brake_Pressure: now also R37.1, R40.1; no longer J2.17 (Pin_17)
- net GND: now also R35.2, R36.2, R37.2, R38.2, R39.2, R45.2, R47.2, R49.2
- net SUS1: now also R38.1, R41.1; no longer J2.21 (Pin_21)
- net SUS2: now also R39.1, R42.1; no longer J2.20 (Pin_20)
- net SUS3: now also R35.1, R43.1; no longer J2.19 (Pin_19)
- net SUS4: now also R36.1, R44.1; no longer J2.18 (Pin_18)
- new net A2: J2.16 (Pin_16), R46.2
- new net A3: J2.15 (Pin_15), R48.2
- new net A4: J2.14 (Pin_14), R50.2
- new net BRK_P: J2.17 (Pin_17), R40.2
- new net SUSP1: J2.21 (Pin_21), R41.2
- new net SUSP2: J2.20 (Pin_20), R42.2
- new net SUSP3: J2.19 (Pin_19), R43.2
- new net SUSP4: J2.18 (Pin_18), R44.2

Commit message: vcu fix
Parts:
- removed R35, R36, R37, R38, R39, R45, R47, R49: 2K, Resistor_SMD:R_0402_1005Metric_Pad0.72x0.64mm_HandSolder, symbol Device:R
- removed R40, R41, R42, R43, R44, R46, R48, R50: 3K, Resistor_SMD:R_0402_1005Metric_Pad0.72x0.64mm_HandSolder, symbol Device:R
- D10, D11, D12, D3, D4, D9: footprint Diode_SMD:D_0603_1608Metric_Pad1.05x0.95mm_HandSolder -> Diode_SMD:D_SOD-123

Commit message: tambah i2c di tele
Connections:
- net Ac2 is gone; now on net A2: U2.8 (A1)
- net Ac3 is gone; now on net A3: U2.9 (A2)
- net Ac4 is gone; now on net A4: U2.10 (A3)
- net Brake_Pressure is gone; now on net BRK_P: U2.7 (A0)
- net SUS1 is gone; now on net SUSP1: U1.7 (A0)
- net SUS2 is gone; now on net SUSP2: U1.8 (A1)
- net SUS3 is gone; now on net SUSP3: U1.9 (A2)
- net SUS4 is gone; now on net SUSP4: U1.10 (A3)
- net GND: no longer J2.2 (Pin_2), J2.3 (Pin_3)
- net SCL: now also J2.3 (Pin_3)
- net SDA: now also J2.2 (Pin_2)
Changed lines of the file:
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@@
 	(wire
 		(pts
-			(xy 152.4 176.53) (xy 163.83 176.53)
+			(xy 152.4 176.53) (xy 162.56 176.53)
 		)
 		(stroke
@@
 	(wire
 		(pts
-			(xy 152.4 173.99) (xy 161.29 173.99)
+			(xy 152.4 173.99) (xy 162.56 173.99)
 		)
 		(stroke
@@
 		)
 	)
-	(label "Ac3"
+	(label "A3"
 		(at 304.8 45.72 0)
 		(effects
@@
 		)
 	)
-	(label "SUS2"
+	(label "SUSP2"
 		(at 260.35 44.45 0)
 		(effects
@@
 		)
 	)
-	(label "SUS4"
+	(label "SUSP4"
 		(at 260.35 49.53 0)
 		(effects
@@
 		)
 	)
-	(label "Ac2"
+	(label "A2"
 		(at 304.8 43.18 0)
 		(effects
@@
 		)
 	)
+	(label "SCL"
+		(at 162.56 176.53 0)
+		(effects
+			(font
+				(size 1.27 1.27)
+			)
+			(justify left bottom)
+		)
+	)
 	(label "ADR2"
 		(at 271.78 48.26 0)
@@
 		)
 	)
-	(label "SUS3"
+	(label "SUSP3"
 		(at 260.35 46.99 0)
 		(effects
@@
 		)
 	)
+	(label "SDA"
+		(at 162.56 173.99 0)
+		(effects
+			(font
+				(size 1.27 1.27)
+			)
+			(justify left bottom)
+		)
+	)
 	(label "TX_Pneu"
 		(at 278.13 152.4 0)
@@
 		)
 	)
-	(label "Brake_Pressure"
+	(label "BRK_P"
 		(at 304.8 40.64 0)
 		(effects
@@
 		)
 	)
-	(label "SUS1"
+	(label "SUSP1"
 		(at 260.35 41.91 0)
 		(effects
@@
 		)
 	)
-	(label "Ac4"
+	(label "A4"
 		(at 304.8 48.26 0)
 		(effects
@@
 		)
 		(property "Intersheetrefs" "${INTERSHEET_REFS}"
-			(at 167.7828 212.09 0)
+			(at 167.1286 212.09 0)
 			(effects
 				(font
@@
 	)
 	(symbol
-		(lib_id "power:GND")
-		(at 161.29 173.99 90)
-		(unit 1)
-		(exclude_from_sim no)
-		(in_bom yes)
-		(on_board yes)
-		(dnp no)
-		(property "Reference" "#PWR086"
-			(at 167.64 173.99 0)
-			(effects
-				(font
-					(size 1.27 1.27)
-				)
-				(hide yes)
-			)
-		)
-		(property "Value" "GND"
-			(at 164.084 172.72 90)
-			(effects
-				(font
-					(size 1.27 1.27)
-				)
-				(justify right)
-			)
-		)
-		(property "Footprint" ""
-			(at 161.29 173.99 0)
-			(effects
-				(font
-					(size 1.27 1.27)
-				)
-				(hide yes)
-			)
-		)
-		(property "Datasheet" ""
-			(at 161.29 173.99 0)
-			(effects
-				(font
-					(size 1.27 1.27)
-				)
-				(hide yes)
-			)
-		)
-		(property "Description" "Power symbol creates a global label with name \"GND\" , ground"
-			(at 161.29 173.99 0)
-			(effects
-				(font
-					(size 1.27 1.27)
-				)
-				(hide yes)
-			)
-		)
-		(pin "1"
-		)
-		(instances
-			(project "VCU"
-				(path "/f790f722-c1e4-44ca-a34d-198a0a886df2"
-					(reference "#PWR086")
-					(unit 1)
-				)
-			)
-		)
-	)
-	(symbol
 		(lib_id "Device:R_Small_US")
 		(at 60.96 229.87 180)
@@
 					(unit 1)
 				)
-			)
-		)
-	)
-	(symbol
-		(lib_id "power:GND")
-		(at 163.83 176.53 90)
-		(unit 1)
-		(exclude_from_sim no)
-		(in_bom yes)
-		(on_board yes)
-		(dnp no)
-		(property "Reference" "#PWR053"
-			(at 170.18 176.53 0)
-			(effects
-				(font
-					(size 1.27 1.27)
-				)
-				(hide yes)
-			)
-		)
-		(property "Value" "GND"
-			(at 166.624 175.26 90)
-			(effects
-				(font
-					(size 1.27 1.27)
-				)
-				(justify right)
-			)
-		)
-		(property "Footprint" ""
-			(at 163.83 176.53 0)
-			(effects
-				(font
-					(size 1.27 1.27)
-				)
-				(hide yes)
-			)
-		)
-		(property "Datasheet" ""
-			(at 163.83 176.53 0)
-			(effects
-				(font
-					(size 1.27 1.27)
-				)
-				(hide yes)
-			)
-		)
-		(property "Description" "Power symbol creates a global label with name \"GND\" , ground"
-			(at 163.83 176.53 0)
-			(effects
-				(font
-					(size 1.27 1.27)
-				)
-				(hide yes)
-			)
-		)
-		(pin "1"
-		)
-		(instances
-			(project ""
-				(path "/f790f722-c1e4-44ca-a34d-198a0a886df2"
-					(reference "#PWR053")
-					(unit 1)
-				)
