File: Bimasakti BM-13 EVO/PCB/VCU BARUU/VCU.kicad_pcb (KiCad board)
At the start: 2 copper layers, 20 parts, among them Q1 IRLZ44N, Q2 IRLZ44N, Q3 IRLZ44N, U1 Teensy4.1, U2 SN65HVD230, U3 SN65HVD230, U4 ADS1115IDGS, U5 SN65HVD230

Commit message: cicil assembly
Parts:
- removed Q1, Q2, Q3: IRLZ44N, Package_TO_SOT_THT:TO-220-3_Vertical
- added C2: 0.1uF, Capacitor_SMD:C_0603_1608Metric, F.Cu at (134.0, 84.4)
- added J1: 6437288-3, 0_VCU_CONNECTOR_TE_6437288-3:VCU_CONNECTOR_TE_6437288-3, F.Cu at (132.0, 9.25)
- added R12: 5k, Resistor_SMD:R_0805_2012Metric, F.Cu at (167.6, 79.8)
- added R13: 5k, Resistor_SMD:R_0805_2012Metric, F.Cu at (167.6, 82.7)
- added R14: 5k, Resistor_SMD:R_0805_2012Metric, F.Cu at (167.6, 85.7)
- added R15: 5k, Resistor_SMD:R_0805_2012Metric, F.Cu at (167.6, 88.6)
- added R16: 10K, Resistor_SMD:R_0805_2012Metric, F.Cu at (129.8, 84.6)
- added R17: 10K, Resistor_SMD:R_0805_2012Metric, F.Cu at (129.8, 87.5)
- added U10: ~, Package_TO_SOT_SMD:TO-252-2, F.Cu at (160.1, 115.3)
- added U11: ADS1115IDGS, Package_SO:TSSOP-10_3x3mm_P0.5mm, F.Cu at (131.1, 80.8)
- added U6: ~, Package_TO_SOT_SMD:TO-252-2, F.Cu at (160.1, 82.5)
- added U7: ~, Package_TO_SOT_SMD:TO-252-2, F.Cu at (160.1, 90.7)
- added U8: ~, Package_TO_SOT_SMD:TO-252-2, F.Cu at (160.1, 98.9)
- added U9: ~, Package_TO_SOT_SMD:TO-252-2, F.Cu at (160.1, 107.1)
- R10, R11, R9: value 1K -> 5k
- moved U1 47.5 mm to (103.1, 100.5), turned to 90 degrees
Connections:
- U1 pad 1: unconnected-(U1-GND-Pad1) -> GND
- U1 pad 46: unconnected-(U1-3V3-Pad46) -> 3V3
- U4 pad 4: unconnected-(U4-AIN0-Pad4) -> SUSP1
- U4 pad 5: unconnected-(U4-AIN1-Pad5) -> SUSP2
- U4 pad 6: unconnected-(U4-AIN2-Pad6) -> SUSP3
- U4 pad 7: unconnected-(U4-AIN3-Pad7) -> SUSP4
Other:
- board outline added: 283 x 196.1 mm

Commit message: buat placeholder baru dan ganti konektor
Parts:
- removed C1, C2: 0.1uF, Capacitor_SMD:C_0603_1608Metric
- removed R1, R2, R3, R4, R7, R8: R, Resistor_SMD:R_0805_2012Metric
- removed R10, R11, R12, R13, R14, R15, R9: 5k, Resistor_SMD:R_0805_2012Metric
- removed R16, R17, R5, R6: 10K, Resistor_SMD:R_0805_2012Metric
- removed U1: Teensy4.1, Teensy:Teensy41
- removed U10, U6, U7, U8, U9: ~, Package_TO_SOT_SMD:TO-252-2
- removed U11, U4: ADS1115IDGS, Package_SO:TSSOP-10_3x3mm_P0.5mm
- removed U2, U3, U5: SN65HVD230, Package_SO:SOIC-8_3.9x4.9mm_P1.27mm
- added J2: 12V, Connector_JST:JST_XH_B2B-XH-A_1x02_P2.50mm_Vertical, F.Cu at (73.0, 73.3)
- added J3: 3V3_1, Connector_JST:JST_XH_B2B-XH-A_1x02_P2.50mm_Vertical, F.Cu at (73.0, 83.8)
- added J4: 3V3_2, Connector_JST:JST_XH_B2B-XH-A_1x02_P2.50mm_Vertical, F.Cu at (73.0, 92.7)
- added J5: 5V_1, Connector_JST:JST_XH_B2B-XH-A_1x02_P2.50mm_Vertical, F.Cu at (73.0, 121.4)
- added J6: 5V_2, Connector_JST:JST_XH_B2B-XH-A_1x02_P2.50mm_Vertical, F.Cu at (73.0, 112.7)
- added J7: 5V_3, Connector_JST:JST_XH_B2B-XH-A_1x02_P2.50mm_Vertical, F.Cu at (73.0, 103.7)
- added J8: Conn_02x06_Top_Bottom, Connector_Molex:Molex_Nano-Fit_105310-xx12_2x06_P2.50mm_Vertical, F.Cu at (71.7, 183.9)
- moved J1 229.2 mm to (123.5, 238.3), turned to 0 degrees
Connections:
- J1 pad 13: 12V -> unconnected-(J1-Pad13)
Other:
- board size 283 x 196.1 mm -> 191.5 x 184.9 mm

Commit message: assembly kurang pneumatic, kurang wiring dudukan motherboard
Parts:
- added BSPD1: ~, 0_FootPrintBPSD:FootPrintBPSD, F.Cu at (289.6, 146.8)
- added J10: Conn_01x02_Socket, Connector_Molex:Molex_Nano-Fit_105309-xx02_1x02_P2.50mm_Vertical, F.Cu at (156.3, 263.6)
- added J9: SIGNAL 2, Connector_Molex:Molex_Nano-Fit_105310-xx12_2x06_P2.50mm_Vertical, F.Cu at (156.5, 228.9)
- added U1: ~, 0_FootprintTelemetry:0_FootprintTelemetry, F.Cu at (206.6, 147.1)
- added U2: ~, 0_FootprintVCU:FootprintVCU, F.Cu at (209.1, 236.4)
- J8: value Conn_02x06_Top_Bottom -> SIGNAL 1
- moved J8 105.1 mm to (156.4, 246.2)
- moved J1 103.6 mm to (202.8, 305.0)
- moved J3 92.7 mm to (154.3, 128.3)
- moved J4 92.7 mm to (154.3, 137.2)
- moved J5 92.7 mm to (154.3, 165.9)
- moved J6 92.7 mm to (154.3, 157.1)
- moved J7 92.7 mm to (154.3, 148.2)
- moved J2 92.7 mm to (154.3, 117.8)
Connections:
- J1 pad 18: unconnected-(J1-Pad18) -> COM_BSPD
- J1 pad 19: unconnected-(J1-Pad19) -> NC_BSPD
- J1 pad 2: BRK_LIGHT -> BRAKE_LIGHT
- J1 pad 20: unconnected-(J1-Pad20) -> ECU_HI
- J1 pad 21: unconnected-(J1-Pad21) -> ECU_LO
- J1 pad 22: unconnected-(J1-Pad22) -> BMS_HI
- J1 pad 23: unconnected-(J1-Pad23) -> BMS_LO
- J1 pad 24: unconnected-(J1-Pad24) -> DISP_HI
- J1 pad 25: unconnected-(J1-Pad25) -> DISP_LO
- J1 pad 32: unconnected-(J1-Pad32) -> SDC_IN
- J1 pad 33: unconnected-(J1-Pad33) -> SDC_OUT
- J1 pad 35: ESC_CAN1 -> ESC1_HI
- J1 pad 36: ESC_CAN2 -> ESC1_LO
- J1 pad 37: WS1 -> ESC2_HI
- J1 pad 38: WS2 -> ESC2_LO
- J1 pad 39: WS3 -> WS1
- J1 pad 4: AIR -> unconnected-(J1-Pad4)
- J1 pad 40: WS4 -> unconnected-(J1-Pad40)
- J1 pad 41: APPS1 -> unconnected-(J1-Pad41)
- J1 pad 42: APPS2 -> unconnected-(J1-Pad42)
- J1 pad 43: STEER -> unconnected-(J1-Pad43)
- J1 pad 44: GPOS -> unconnected-(J1-Pad44)
- J1 pad 48: unconnected-(J1-Pad48) -> FAN_BATT
- J1 pad 5: SWITCH_HY -> unconnected-(J1-Pad5)
- J1 pad 52: unconnected-(J1-Pad52) -> SAFETY
- J1 pad 56: unconnected-(J1-Pad56) -> SWITCH_HY
- J1 pad 57: unconnected-(J1-Pad57) -> AIR
- J1 pad 58: unconnected-(J1-Pad58) -> SAFETY
- J1 pad 59: unconnected-(J1-Pad59) -> PDM
- J1 pad 6: ENG_RLY -> unconnected-(J1-Pad6)
- J1 pad 60: unconnected-(J1-Pad60) -> ENGINE
- J8 pad 1: unconnected-(J8-Pin_1-Pad1) -> SCK
- J8 pad 10: unconnected-(J8-Pin_10-Pad10) -> STEER_IN
- J8 pad 11: unconnected-(J8-Pin_11-Pad11) -> APPS_IN2
- J8 pad 12: unconnected-(J8-Pin_12-Pad12) -> APPS_IN1
- J8 pad 2: unconnected-(J8-Pin_2-Pad2) -> MISO
- J8 pad 3: unconnected-(J8-Pin_3-Pad3) -> MOSI
- J8 pad 4: unconnected-(J8-Pin_4-Pad4) -> SS
- J8 pad 5: unconnected-(J8-Pin_5-Pad5) -> STM_TX
- J8 pad 6: unconnected-(J8-Pin_6-Pad6) -> STM_RX
- J8 pad 7: unconnected-(J8-Pin_7-Pad7) -> GND
- J8 pad 8: unconnected-(J8-Pin_8-Pad8) -> ESC1_LO
- J8 pad 9: unconnected-(J8-Pin_9-Pad9) -> ESC1_HI
Routing:
- net AIR: track 0.00 -> 154.5 mm
- net SWITCH_HY: track 0.00 -> 143.5 mm, vias 0 -> 4
- net PDM: track 0.00 -> 141.7 mm
- net ENGINE: track 0.00 -> 124.7 mm
- net SAFETY: track 0.00 -> 3.12 mm
Other:
- board size 191.5 x 184.9 mm -> 180 x 210 mm
