File: Bimasakti BM-13 EVO/PCB/Pneumatic/Pneumatic/Pneumatic.kicad_sch (KiCad schematic)
At the start: 17 parts, among them J1 Conn_01x20_Pin, J2 Conn_01x20_Pin, Q5 DMTH6004SK3, Q6 DMTH6004SK3, U3 YAAJ_BluePill_SWD_Breakout, U7 TCMT1103, U8 TCMT1103

Commit message: assembly VCU FINISH!!!
Parts:
- added D8: LED, LED_SMD:LED_0603_1608Metric_Pad1.05x0.95mm_HandSolder, symbol Device:LED
- added R30: 1K, Resistor_SMD:R_0603_1608Metric_Pad0.98x0.95mm_HandSolder, symbol Device:R_Small_US
Connections:
- net +5V: now also R30.1
- net GND: now also J1.10 (Pin_10), J1.13 (Pin_13), J1.17 (Pin_17), J1.18 (Pin_18), J1.19 (Pin_19), J1.20 (Pin_20), J1.7 (Pin_7), J2.10 (Pin_10), J2.11 (Pin_11), J2.12 (Pin_12), J2.13 (Pin_13), J2.14 (Pin_14), J2.15 (Pin_15), J2.16 (Pin_16), J2.17 (Pin_17), J2.18 (Pin_18), J2.19 (Pin_19), J2.2 (Pin_2), J2.3 (Pin_3), J2.4 (Pin_4), J2.5 (Pin_5), J2.6 (Pin_6), J2.7 (Pin_7), J2.8 (Pin_8), D8.1 (K)
- new net: D8.2 (A), R30.2
