File: Bimasakti BM-13 EVO/PCB/Pneumatic/Pneumatic/Pneumatic.kicad_pcb (KiCad board)
At the start: 2 copper layers, 62 x 68 mm, 22 parts, among them J1 Conn_01x20_Pin, J2 Conn_01x20_Pin, Q5 DMTH6004SK3, Q6 DMTH6004SK3, U3 YAAJ_BluePill_SWD_Breakout, U7 TCMT1103, U8 TCMT1103

Commit message: assembly VCU FINISH!!!
Parts:
- added D8: LED, LED_SMD:LED_0603_1608Metric_Pad1.05x0.95mm_HandSolder, F.Cu at (127.0, 62.9)
- added R30: 1K, Resistor_SMD:R_0603_1608Metric_Pad0.98x0.95mm_HandSolder, F.Cu at (134.7, 65.5)
Connections:
- J1 pad 10: unconnected-(J1-Pin_10-Pad10) -> GND
- J1 pad 13: unconnected-(J1-Pin_13-Pad13) -> GND
- J1 pad 17: unconnected-(J1-Pin_17-Pad17) -> GND
- J1 pad 18: unconnected-(J1-Pin_18-Pad18) -> GND
- J1 pad 19: unconnected-(J1-Pin_19-Pad19) -> GND
- J1 pad 20: unconnected-(J1-Pin_20-Pad20) -> GND
- J1 pad 7: unconnected-(J1-Pin_7-Pad7) -> GND
- J2 pad 10: unconnected-(J2-Pin_10-Pad10) -> GND
- J2 pad 11: unconnected-(J2-Pin_11-Pad11) -> GND
- J2 pad 12: unconnected-(J2-Pin_12-Pad12) -> GND
- J2 pad 13: unconnected-(J2-Pin_13-Pad13) -> GND
- J2 pad 14: unconnected-(J2-Pin_14-Pad14) -> GND
- J2 pad 15: unconnected-(J2-Pin_15-Pad15) -> GND
- J2 pad 16: unconnected-(J2-Pin_16-Pad16) -> GND
- J2 pad 17: unconnected-(J2-Pin_17-Pad17) -> GND
- J2 pad 18: unconnected-(J2-Pin_18-Pad18) -> GND
- J2 pad 19: unconnected-(J2-Pin_19-Pad19) -> GND
- J2 pad 2: unconnected-(J2-Pin_2-Pad2) -> GND
- J2 pad 3: unconnected-(J2-Pin_3-Pad3) -> GND
- J2 pad 4: unconnected-(J2-Pin_4-Pad4) -> GND
- J2 pad 5: unconnected-(J2-Pin_5-Pad5) -> GND
- J2 pad 6: unconnected-(J2-Pin_6-Pad6) -> GND
- J2 pad 7: unconnected-(J2-Pin_7-Pad7) -> GND
- J2 pad 8: unconnected-(J2-Pin_8-Pad8) -> GND
Routing:
- net Net-(D8-A): track 0.00 -> 11.5 mm, vias 0 -> 2
- net +5V: track 51.5 -> 57.2 mm, vias 0 -> 1
- net GND: vias 52 -> 55
Other:
- board text added: "ARJUN GAY"

Commit message: update
Parts:
- renumbered D8 to LED
Changed lines of the file:
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@@
 		(tags "module BlluePill Blue Pill header SWD breakout")
 		(property "Reference" "U3"
-			(at 7.62 -3.81 0)
+			(at 8.3065 -0.0445 0)
 			(layer "F.SilkS")
 			(effects
@@
 		(descr "LED SMD 0603 (1608 Metric), square (rectangular) end terminal, IPC-7351 nominal, (Body size source: http://www.tortai-tech.com/upload/download/2011102023233369053.pdf), generated with kicad-footprint-generator")
 		(tags "LED handsolder")
-		(property "Reference" "D8"
-			(at 0 -1.43 90)
+		(property "Reference" "LED"
+			(at -0.044143 1.685427 90)
 			(layer "F.SilkS")
 			(effects
