File: Bimasakti BM-13 EVO/PCB/Torque Vectoring Board/Torque Vectoring Board.kicad_sch (KiCad schematic)
At the start: 34 parts, among them J1 SIGNAL 1, J2 SIGNAL 2, J3 wsout1, J4 wsout2, U3 SN65HVD230, U4 SN65HVD230, U5 ADS1115IDGS

Commit message: update tv board
Connections:
- net GND: no longer U6.25 (RX), U6.26 (GND), U6.27 (TX), U6.29 (SCL), U6.31 (SDA), U6.4 (WS_FR_OUT), U6.5 (WS_FL_OUT), U6.6 (WS_RR_OUT), U6.7 (WS_RL_OUT)
- net SCL: now also U6.29 (SCL)
- net SDA: now also U6.31 (SDA)
- net STM_RX: now also U6.25 (RX)
- net STM_TX: now also U6.27 (TX)
- net WS_RRo: now reaches J4.1 (Pin_1)
- net WS_RRo: now also U6.6 (WS_RR_OUT)
- net WS_RLo: now reaches J4.2 (Pin_2)
- net WS_RLo: now also U6.7 (WS_RL_OUT)
- net WS_FRo: now reaches J3.1 (Pin_1)
- net WS_FRo: now also U6.4 (WS_FR_OUT)
- net WS_FLo: now reaches J3.2 (Pin_2)
- net WS_FLo: now also U6.5 (WS_FL_OUT)
- net GPOS: no longer names the net of U1.72 (PA6)

Commit message: pdm and tv fix
Parts:
- removed U6: ~, 0_CUSTOM_PCB:wheelspeed, symbol 0_CUSTOM_PCB:Wheelspeed
- added U6: ~, 0_WHEELSPEED:Untitled, symbol 0_wheelspeed:wheelspeed
- J3, J4: footprint TerminalBlock_Phoenix:TerminalBlock_Phoenix_PT-1,5-2-5.0-H_1x02_P5.00mm_Horizontal -> Connector_Molex:Molex_Nano-Fit_105309-xx02_1x02_P2.50mm_Vertical
- R10, R11, R12, R13, R14, R15, R2, R3, R4, R5, R6, R7, R8, R9: footprint Resistor_SMD:R_0805_2012Metric -> Resistor_SMD:R_0603_1608Metric
Connections:
- net 12V: now also U6.2 (12V)
- net 5V: now also U6.1 (5V)
- net CAN1_RX: now also U1.21 (PA11/USBM); no longer U1.24 (PA12/USB_DP)
- net CAN1_TX: now also U1.24 (PA12/USB_DP); no longer U1.21 (PA11/USBM)
- net CAN2_RX: now also U1.54 (PB12); no longer U1.53 (PB13)
- net CAN2_TX: now also U1.53 (PB13); no longer U1.54 (PB12)
- net GND: now also J2.1 (Pin_1), J2.12 (Pin_12), J2.6 (Pin_6), J2.7 (Pin_7), J2.8 (Pin_8), J2.9 (Pin_9), U6.15 (GND)
- net SCL: now also U6.14 (SCL)
- net SDA: now also U6.13 (SDA)
- net STM_RX: now also U6.4 (TX); no longer J1.6 (Pin_6)
- net STM_TX: now also U6.3 (RX); no longer J1.5 (Pin_5)
- net WS_FL: now also U6.8 (WS_FL)
- net WS_FLo: now also U6.11 (WS_FR_O)
- net WS_FR: now also U6.7 (WS_FR)
- net WS_FRo: now also U6.12 (WS_FL_O)
- net WS_RL: now also U6.6 (WS_RL)
- net WS_RLo: now also U6.9 (WS_RL_O)
- net WS_RR: now also U6.5 (WS_RR)
- net WS_RRo: now also U6.10 (WS_RR_O)
- net STM_TX_2: now reaches U1.28 (PC12)
- net STM_TX_2: now also J1.5 (Pin_5)
- net STM_RX_2: now reaches U1.29 (PD2)
- net STM_RX_2: now also J1.6 (Pin_6)

Commit message: tv board FIXXXXX
Connections:
- net WS_FLo: now also J3.1 (Pin_1), U1.43 (PE1), U6.12 (WS_FL_O); no longer J3.2 (Pin_2), U6.11 (WS_FR_O)
- net WS_FRo: now also J3.2 (Pin_2), U1.41 (PB9), U6.11 (WS_FR_O); no longer J3.1 (Pin_1), U6.12 (WS_FL_O)
- net WS_RLo: now also U1.35 (PB3)
- net WS_RRo: now also U1.37 (PB5)

Commit message: kontol tadi ga kesave
Connections:
- net WS_FL: now also U6.7 (WS_FL); no longer U6.8 (WS_FL)
- net WS_FLo: now also J3.2 (Pin_2), U1.41 (PB9); no longer J3.1 (Pin_1), U1.43 (PE1)
- net WS_FR: now also U6.8 (WS_FR); no longer U6.7 (WS_FR)
- net WS_FRo: now also J3.1 (Pin_1), U1.43 (PE1); no longer J3.2 (Pin_2), U1.41 (PB9)
Changed lines of the file:
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@@
 	(wire
 		(pts
-			(xy 217.17 80.01) (xy 219.71 80.01)
+			(xy 90.17 133.35) (xy 91.44 133.35)
 		)
 		(stroke
@@
 	(wire
 		(pts
-			(xy 215.9 66.04) (xy 218.44 66.04)
+			(xy 217.17 80.01) (xy 219.71 80.01)
 		)
 		(stroke
@@
 	(wire
 		(pts
-			(xy 209.55 139.7) (xy 217.17 139.7)
+			(xy 215.9 68.58) (xy 218.44 68.58)
 		)
 		(stroke
@@
 	(wire
 		(pts
-			(xy 106.68 171.45) (xy 109.22 171.45)
+			(xy 209.55 139.7) (xy 217.17 139.7)
 		)
 		(stroke
@@
 	(wire
 		(pts
-			(xy 134.62 110.49) (xy 137.16 110.49)
+			(xy 106.68 171.45) (xy 109.22 171.45)
 		)
 		(stroke
@@
 	(wire
 		(pts
-			(xy 90.17 138.43) (xy 91.44 138.43)
+			(xy 134.62 110.49) (xy 137.16 110.49)
 		)
 		(stroke
@@
 	(wire
 		(pts
-			(xy 90.17 133.35) (xy 91.44 133.35)
-		)
-		(stroke
-			(width 0)
-			(type default)
-		)
-	)
-	(wire
-		(pts
 			(xy 134.62 120.65) (xy 139.7 120.65)
 		)
@@
 	(wire
 		(pts
+			(xy 215.9 66.04) (xy 218.44 66.04)
+		)
+		(stroke
+			(width 0)
+			(type default)
+		)
+	)
+	(wire
+		(pts
 			(xy 229.87 114.3) (xy 229.87 116.84)
 		)
@@
 	(wire
 		(pts
-			(xy 256.54 46.99) (xy 256.54 49.53)
-		)
-		(stroke
-			(width 0)
-			(type default)
-		)
-	)
-	(wire
-		(pts
 			(xy 77.47 25.4) (xy 77.47 29.21)
 		)
@@
 	(wire
 		(pts
+			(xy 256.54 46.99) (xy 256.54 49.53)
+		)
+		(stroke
+			(width 0)
+			(type default)
+		)
+	)
+	(wire
+		(pts
 			(xy 69.85 118.11) (xy 69.85 119.38)
 		)
@@
 	(wire
 		(pts
+			(xy 90.17 138.43) (xy 91.44 138.43)
+		)
+		(stroke
+			(width 0)
+			(type default)
+		)
+	)
+	(wire
+		(pts
 			(xy 39.37 83.82) (xy 41.91 83.82)
 		)
@@
 	(wire
 		(pts
-			(xy 215.9 68.58) (xy 218.44 68.58)
-		)
-		(stroke
-			(width 0)
-			(type default)
-		)
-	)
-	(wire
-		(pts
 			(xy 222.25 80.01) (xy 224.79 80.01)
 		)
@@
 	(global_label "WS_FRo"
 		(shape input)
-		(at 256.54 49.53 270)
+		(at 254 49.53 270)
 		(fields_autoplaced yes)
 		(effects
@@
 		)
 		(property "Intersheetrefs" "${INTERSHEET_REFS}"
-			(at 256.54 59.6513 90)
+			(at 254 59.6513 90)
 			(effects
 				(font
@@
 	(global_label "WS_FL"
 		(shape input)
-		(at 215.9 68.58 180)
+		(at 215.9 66.04 180)
 		(fields_autoplaced yes)
 		(effects
@@
 		)
 		(property "Intersheetrefs" "${INTERSHEET_REFS}"
-			(at 207.1696 68.58 0)
+			(at 207.1696 66.04 0)
 			(effects
 				(font
@@
 	(global_label "WS_FLo"
 		(shape input)
-		(at 90.17 138.43 180)
+		(at 90.17 133.35 180)
 		(fields_autoplaced yes)
 		(effects
@@
 		)
 		(property "Intersheetrefs" "${INTERSHEET_REFS}"
-			(at 80.2906 138.43 0)
+			(at 80.2906 133.35 0)
 			(effects
 				(font
@@
 	(global_label "WS_FR"
 		(shape input)
-		(at 215.9 66.04 180)
+		(at 215.9 68.58 180)
 		(fields_autoplaced yes)
 		(effects
@@
 		)
 		(property "Intersheetrefs" "${INTERSHEET_REFS}"
-			(at 206.9277 66.04 0)
+			(at 206.9277 68.58 0)
 			(effects
 				(font
@@
 	(global_label "WS_FLo"
 		(shape input)
-		(at 254 49.53 270)
+		(at 256.54 49.53 270)
 		(fields_autoplaced yes)
 		(effects
@@
 		)
 		(property "Intersheetrefs" "${INTERSHEET_REFS}"
-			(at 254 59.4094 90)
+			(at 256.54 59.4094 90)
 			(effects
 				(font
@@
 	(global_label "WS_FRo"
 		(shape input)
-		(at 90.17 133.35 180)
+		(at 90.17 138.43 180)
 		(fields_autoplaced yes)
 		(effects
@@
 		)
 		(property "Intersheetrefs" "${INTERSHEET_REFS}"
-			(at 80.0487 133.35 0)
+			(at 80.0487 138.43 0)
 			(effects
 				(font

Commit message: gerber tapi gada drillnya blog
Connections:
- net WS_FL: now also U6.8 (WS_FL); no longer U6.7 (WS_FL)
- net WS_FR: now also U6.7 (WS_FR); no longer U6.8 (WS_FR)
Changed lines of the file:
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@@
+	(wire
+		(pts
+			(xy 215.9 66.04) (xy 218.44 66.04)
+		)
+		(stroke
+			(width 0)
+			(type default)
+		)
+	)
 	(wire
 		(pts
@@
 		)
 		(stroke
-			(width 0)
-			(type default)
-		)
-	)
-	(wire
-		(pts
-			(xy 215.9 66.04) (xy 218.44 66.04)
-		)
-		(stroke
