File: Bimasakti BM-13 EVO/PCB/Torque Vectoring Board/Torque Vectoring Board.kicad_pcb (KiCad board)
At the start: 2 copper layers, 99 x 108 mm, 38 parts, among them J1 SIGNAL 1, J2 SIGNAL 2, J3 wsout1, J4 wsout2, U3 SN65HVD230, U4 SN65HVD230, U5 ADS1115IDGS

Commit message: tv board FIXXXXX
Routing:
- net WS_FLo: track 58.6 -> 92.5 mm
- net WS_FRo: track 65.0 -> 87.5 mm
- net STM_RX_2: track 84.7 -> 83.6 mm
Changed lines of the file:
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@@
-	)
-	(segment
-		(start 96.262644 87.122)
-		(end 96.262644 86.553184)
-		(width 0.35)
-		(layer "B.Cu")
-		(net 51)
 	)
 	(segment
@@
 	)
 	(segment
-		(start 96.262644 87.122)
-		(end 96.262644 86.617356)
-		(width 0.35)
-		(layer "B.Cu")
-		(net 51)
-	)
-	(segment
 		(start 99.568 109.728)
 		(end 100.076 109.22)
-		(width 0.35)
-		(layer "B.Cu")
-		(net 51)
-	)
-	(segment
-		(start 96.262644 86.617356)
-		(end 96.266 86.614)
 		(width 0.35)
 		(layer "B.Cu")
@@
 	)
 	(segment
+		(start 112 46.25)
+		(end 106.595 40.845)
+		(width 0.508)
+		(layer "F.Cu")
+		(net 113)
+	)
+	(segment
+		(start 93.5 44.07369)
+		(end 93.5 44.515)
+		(width 0.508)
+		(layer "F.Cu")
+		(net 113)
+	)
+	(segment
+		(start 96.72869 40.845)
+		(end 93.5 44.07369)
+		(width 0.508)
+		(layer "F.Cu")
+		(net 113)
+	)
+	(segment
 		(start 120.396 93.98)
 		(end 112 85.584)
@@
 	(segment
 		(start 112 85.584)
+		(end 112 46.25)
+		(width 0.508)
+		(layer "F.Cu")
+		(net 113)
+	)
+	(segment
+		(start 106.595 40.845)
+		(end 96.72869 40.845)
+		(width 0.508)
+		(layer "F.Cu")
+		(net 113)
+	)
+	(segment
+		(start 112 46.25)
 		(end 112 44)
 		(width 0.508)
 		(layer "F.Cu")
 		(net 113)
+	)
+	(segment
+		(start 91.061948 39.343)
+		(end 88.5 41.904948)
+		(width 0.508)
+		(layer "F.Cu")
+		(net 114)
 	)
 	(segment
@@
 	)
 	(segment
+		(start 88.5 41.904948)
+		(end 88.5 42)
+		(width 0.508)
+		(layer "F.Cu")
+		(net 114)
+	)
+	(segment
+		(start 111.843 39.343)
+		(end 91.061948 39.343)
+		(width 0.508)
+		(layer "F.Cu")
+		(net 114)
+	)
+	(segment
 		(start 118 44.5)
 		(end 116.5 43)
@@
 	)
 	(segment
+		(start 88.5 42)
+		(end 89.727 43.227)
+		(width 0.508)
+		(layer "F.Cu")
+		(net 114)
+	)
+	(segment
 		(start 116.5 43)
 		(end 115.5 43)
@@
 	)
 	(segment
+		(start 89.727 43.227)
+		(end 89.727 45.75)
+		(width 0.508)
+		(layer "F.Cu")
+		(net 114)
+	)
+	(segment
 		(start 118 84.5)
 		(end 118 44.5)
 		(width 0.508)
 		(layer "F.Cu")
+		(net 114)
+	)
+	(segment
+		(start 115.5 43)
+		(end 111.843 39.343)
+		(width 0.508)
+		(layer "F.Cu")

Commit message: kontol tadi ga kesave
Connections:
- U1 pad 35: unconnected-(U1-PB3-Pad35) -> WS_RLo
- U1 pad 37: unconnected-(U1-PB5-Pad37) -> WS_RRo
- U1 pad 41: unconnected-(U1-PB9-Pad41) -> WS_FLo
- U1 pad 43: unconnected-(U1-PE1-Pad43) -> WS_FRo
- U6 pad 11: WS_FLo -> WS_FRo
- U6 pad 12: WS_FRo -> WS_FLo
- U6 pad 7: WS_FR -> WS_FL
- U6 pad 8: WS_FL -> WS_FR
Routing:
- net WS_RLo: track 46.9 -> 90.4 mm
- net WS_RRo: track 51.4 -> 91.6 mm
- net 12V: track 205.2 -> 216.4 mm
- net WS_FLo: track 92.5 -> 84.0 mm
- net WS_FRo: track 87.5 -> 85.7 mm
- net SDA: track 106.2 -> 107.6 mm
- net GND: vias 166 -> 159

Commit message: gerber tapi gada drillnya blog
Connections:
- U6 pad 7: WS_FL -> WS_FR
- U6 pad 8: WS_FR -> WS_FL
Routing:
- net WS_FL: track 71.1 -> 74.5 mm
Changed lines of the file:
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@@
 			(outputformat 1)
 			(mirror no)
-			(drillshape 1)
+			(drillshape 0)
 			(scaleselection 1)
-			(outputdirectory "")
+			(outputdirectory "JLC/")
 		)
 	)
@@
 			(layers "*.Cu" "*.Mask")
 			(remove_unused_layers no)
-			(net 105 "WS_FL")
-			(pinfunction "WS_FL")
+			(net 106 "WS_FR")
+			(pinfunction "WS_FR")
 			(pintype "input")
 		)
@@
 			(layers "*.Cu" "*.Mask")
 			(remove_unused_layers no)
-			(net 106 "WS_FR")
-			(pinfunction "WS_FR")
+			(net 105 "WS_FL")
+			(pinfunction "WS_FL")
 			(pintype "input")
 		)
@@
 	)
 	(segment
-		(start 114.5 136.5)
-		(end 117.856 133.144)
+		(start 114.3 105.8)
+		(end 114.3 103.378)
 		(width 0.35)
 		(layer "B.Cu")
@@
 	)
 	(segment
-		(start 103.054053 98.817983)
-		(end 103.054053 100.197717)
+		(start 108.814338 97.892338)
+		(end 102.357662 97.892338)
 		(width 0.35)
 		(layer "B.Cu")
@@
 	)
 	(segment
-		(start 117.856 133.144)
-		(end 117.856 109.356)
+		(start 114.5 136.5)
+		(end 117.856 133.144)
 		(width 0.35)
 		(layer "B.Cu")
@@
 	)
 	(segment
-		(start 103.054053 100.197717)
-		(end 104.55125 101.694914)
+		(start 99.832 133.048)
+		(end 99.832 135.832)
 		(width 0.35)
 		(layer "B.Cu")
@@
 	)
 	(segment
-		(start 99.832 135.832)
-		(end 100.5 136.5)
+		(start 101.75 101.25)
+		(end 102.194914 101.694914)
 		(width 0.35)
 		(layer "B.Cu")
@@
 	)
 	(segment
-		(start 99.832 133.048)
-		(end 99.832 135.832)
+		(start 100.5 136.5)
+		(end 114.5 136.5)
 		(width 0.35)
 		(layer "B.Cu")
@@
 	)
 	(segment
-		(start 114.3 103.378)
-		(end 108.80685 97.88485)
+		(start 101.75 98.5)
+		(end 101.75 101.25)
 		(width 0.35)
 		(layer "B.Cu")
@@
 	)
 	(segment
-		(start 100.5 136.5)
-		(end 114.5 136.5)
+		(start 117.856 133.144)
+		(end 117.856 109.356)
 		(width 0.35)
 		(layer "B.Cu")
@@
 	)
 	(segment
-		(start 114.3 105.8)
-		(end 114.3 103.378)
+		(start 102.357662 97.892338)
+		(end 101.75 98.5)
 		(width 0.35)
 		(layer "B.Cu")
@@
 	)
 	(segment
-		(start 103.987186 97.88485)
-		(end 103.054053 98.817983)
+		(start 99.832 135.832)
+		(end 100.5 136.5)
 		(width 0.35)
 		(layer "B.Cu")
@@
 	)
 	(segment
-		(start 108.80685 97.88485)
-		(end 103.987186 97.88485)
+		(start 117.856 109.356)
+		(end 114.3 105.8)
 		(width 0.35)
 		(layer "B.Cu")
@@
 	)
 	(segment
-		(start 117.856 109.356)
-		(end 114.3 105.8)
+		(start 102.194914 101.694914)
+		(end 104.55125 101.694914)
+		(width 0.35)
+		(layer "B.Cu")
+		(net 105)
+	)
+	(segment
+		(start 114.3 103.378)
+		(end 108.814338 97.892338)
 		(width 0.35)
 		(layer "B.Cu")
@@
 	)
 	(segment
-		(start 111.506 104.14)
-		(end 106.520914 99.154914)
+		(start 107.154914 99.154914)
+		(end 104.55125 99.154914)
 		(width 0.508)
 		(layer "B.Cu")
@@
 	)
 	(segment
-		(start 111.506 113.316)
-		(end 111.506 104.14)
+		(start 104.284 135)
+		(end 112 135)
 		(width 0.508)
 		(layer "B.Cu")
@@
 	)
 	(segment
-		(start 112 135)
-		(end 113.268 133.732)
+		(start 113.268 115.078)
+		(end 111.506 113.316)
 		(width 0.508)
 		(layer "B.Cu")
@@
 	)
 	(segment
-		(start 106.520914 99.154914)
-		(end 104.55125 99.154914)
+		(start 102.332 133.048)
+		(end 104.284 135)
 		(width 0.508)
 		(layer "B.Cu")
@@
 	)
 	(segment
-		(start 102.332 133.048)
-		(end 104.284 135)
+		(start 111.506 113.316)
+		(end 111.506 103.506)
 		(width 0.508)
 		(layer "B.Cu")
@@
 	)
 	(segment
-		(start 104.284 135)
-		(end 112 135)
+		(start 111.506 103.506)
+		(end 107.154914 99.154914)
 		(width 0.508)
 		(layer "B.Cu")
@@
 	)
 	(segment
-		(start 113.268 115.078)
-		(end 111.506 113.316)
+		(start 112 135)
+		(end 113.268 133.732)
 		(width 0.508)
 		(layer "B.Cu")
