File: Bimasakti BM-13 EVO/PCB/Motherboard/VCU-backups/VCU-2025-05-20_235204/VCU.kicad_sch (KiCad schematic)
At the start: 26 parts, among them J1 6437288-3, J10 power, J11 6437288-3, J2 12V, J3 3V3_1, J4 5V_5, J5 5V_1, J6 5V_2, J7 5V_3, J8 SIGNAL 1, J9 SIGNAL 2

Commit message: vcu lebih rapi
Parts:
- removed U4: ~, 0_FootprintTelemetry:0_FootprintTelemetry, symbol 0_FootprintTelemetry:FootprintTelemetry
- added R2: R, Resistor_SMD:R_0603_1608Metric_Pad0.98x0.95mm_HandSolder, symbol Device:R
- added U1: ~, 0_FootprintTelemetry:0_FootprintTelemetry, symbol 0_FootprintTelemetry:FootprintTelemetry
- R3: footprint Resistor_SMD:R_0603_1608Metric_Pad0.98x0.95mm_HandSolder -> BRK_Press
Connections:
- net 5V_T: now also U1.6 (+5V)
- net AIR: now also J1.39; no longer J11.4
- net APPS_IN1: now also J1.55; no longer J1.1
- net APPS_IN2: now also J1.54; no longer J1.2
- net BMS_HI: now also J1.36; no longer J1.59
- net BMS_LO: now also J1.35; no longer J1.60
- net BRAKE_LIGHT: now also J1.2; no longer J11.1
- net BRK_P: now also J1.3; no longer J1.39
- net CS_T: now also U1.10 (CS2)
- net DISP_HI: now also J1.42; no longer J1.53
- net DISP_LO: now also J1.48; no longer J1.47
- net ECU_HI: now also J1.38; no longer J1.57
- net ECU_LO: now also J1.37; no longer J1.58
- net ENG_RLY: now also J11.26; no longer J11.7
- net ESC1_HI: now also J1.26; no longer J1.4
- net ESC1_LO: now also J1.18; no longer J1.5
- net ESC2_HI: now also J1.10; no longer J1.31
- net ESC2_LO: now also J1.1; no longer J1.30
- net FAN_BATT: now also J11.7; no longer J11.10
- net GND: now also J1.5, R2.1, U1.1 (GND), U1.11 (GND), U1.12 (GND), U1.13 (GND), U1.14 (GND), U1.15 (GND), U1.16 (GND), U1.2 (GND), U1.3 (GND), U1.4 (GND), U1.5 (GND)
- net GPOS: now also J1.58; no longer J11.39
- net IND_SWITCH: now also J1.11; no longer J11.18
- net MISO_T: now also U1.8 (MISO2)
- net MOSI_T: now also U1.7 (MOSI2)
- net PDM: now also J11.18; no longer J11.6
- net SAFETY: now also J1.40, J1.46; no longer J11.3
- net SCK_T: now also U1.9 (SCK2)
- net SDC_IN: now also J11.5; no longer J11.2
- net SDC_OUT: now also J11.6; no longer J11.40
- net STEER_IN: now also J1.27; no longer J1.3
- net SUSP1: now also J1.6; no longer J1.35
- net SUSP2: now also J1.7; no longer J1.36
- net SUSP3: now also J1.8; no longer J1.37
- net SUSP4: now also J1.9; no longer J1.38
- net SWITCH_HY: now also J1.41; no longer J11.5
- net TPS: now also J11.10; no longer J11.41
- net UP: now also R2.2
- net WS_FL: now also J11.3; no longer J1.27
- net WS_FR: now also J11.4; no longer J1.26
- net WS_RL: now also J11.1; no longer J1.29
- net WS_RR: now also J11.2; no longer J1.28
- net NC: now reaches J11.8
- net COM: now reaches J11.9
- net BMS_CAN: now reaches J1.21
- new net COM_BSPD: J1.28
- new net NC_BSPD: J1.29
