File: Bimasakti BM-13 EVO/PCB/Torque Vectoring Board/Torque Vectoring Board-backups/Torque Vectoring Board-2025-05-26_014918/Torque Vectoring Board.kicad_sch (KiCad schematic)
At the start: 34 parts, among them J1 SIGNAL 1, J2 SIGNAL 2, J3 wsout1, J4 wsout2, U3 SN65HVD230, U4 SN65HVD230, U5 ADS1115IDGS

Commit message: tv dengan pdm kecil
Parts:
- J3, J4: footprint Connector_Molex:Molex_Nano-Fit_105309-xx02_1x02_P2.50mm_Vertical -> TerminalBlock_Phoenix:TerminalBlock_Phoenix_PT-1,5-2-5.0-H_1x02_P5.00mm_Horizontal
- U6: footprint 0_WHEELSPEED:Untitled -> (none)
Connections:
- net GND: no longer J2.1 (Pin_1), J2.12 (Pin_12), J2.6 (Pin_6), J2.7 (Pin_7), J2.8 (Pin_8), J2.9 (Pin_9)
- net STM_RX: now also J1.6 (Pin_6)
- net STM_TX: now also J1.5 (Pin_5)
- net STM_RX_2: no longer names the net of U1.29 (PD2)
- net STM_RX_2: no longer J1.6 (Pin_6)
- net STM_TX_2: no longer names the net of U1.28 (PC12)
- net STM_TX_2: no longer J1.5 (Pin_5)
