File: Bimasakti BM-13 EVO/PCB/Wheelspeed Module/Wheelspeed New/Wheelspeed New.kicad_sch (KiCad schematic)
At the start: 21 parts, among them J3 Conn_01x15_Pin, J4 Conn_01x15_Pin, U1 ESP32-C3_SUPERMINI_TH, U2 LM393

Commit message: tv board FIXXXXX
Connections:
- net WS_FL_Signal: now also J4.12 (Pin_12)
- net WS_FR_Signal: now also J4.11 (Pin_11)
- net WS_RL_Signal: now also J4.9 (Pin_9)
- net WS_RR_Signal: now also J4.10 (Pin_10)
Changed lines of the file:
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@@
+	(wire
+		(pts
+			(xy 255.27 93.98) (xy 261.62 93.98)
+		)
+		(stroke
+			(width 0)
+			(type default)
+		)
+	)
 	(wire
 		(pts
@@
 	(wire
 		(pts
+			(xy 255.27 99.06) (xy 261.62 99.06)
+		)
+		(stroke
+			(width 0)
+			(type default)
+		)
+	)
+	(wire
+		(pts
 			(xy 226.06 97.79) (xy 231.14 97.79)
 		)
@@
 	(wire
 		(pts
+			(xy 255.27 96.52) (xy 261.62 96.52)
+		)
+		(stroke
+			(width 0)
+			(type default)
+		)
+	)
+	(wire
+		(pts
 			(xy 226.06 87.63) (xy 233.68 87.63)
 		)
@@
 		(pts
 			(xy 172.72 34.29) (xy 176.53 34.29)
+		)
+		(stroke
+			(width 0)
+			(type default)
+		)
+	)
+	(wire
+		(pts
+			(xy 255.27 91.44) (xy 261.62 91.44)
 		)
 		(stroke
@@
 		)
 	)
+	(label "WS_FR_Signal"
+		(at 261.62 96.52 0)
+		(effects
+			(font
+				(size 1.27 1.27)
+			)
+			(justify left bottom)
+		)
+	)
 	(label "TX"
 		(at 83.82 45.72 0)
@@
 		)
 	)
+	(label "WS_RR_Signal"
+		(at 261.62 93.98 0)
+		(effects
+			(font
+				(size 1.27 1.27)
+			)
+			(justify left bottom)
+		)
+	)
 	(label "RX"
 		(at 233.68 87.63 0)
@@
 		(effects
 			(font
+				(size 1.27 1.27)
+			)
+			(justify left bottom)
+		)
+	)
+	(label "WS_FL_Signal"
+		(at 261.62 99.06 0)
+		(effects
+			(font
+				(size 1.27 1.27)
+			)
+			(justify left bottom)
+		)
+	)
+	(label "WS_RL_Signal"
+		(at 261.62 91.44 0)
+		(effects
+			(font

Commit message: kontol tadi ga kesave
Connections:
- net GND: now also J4.2 (Pin_2), J4.6 (Pin_6), J4.8 (Pin_8)
- net SDA: now reaches U1.8 (GPIO8)
- net SDA: now also J3.1 (Pin_1)
- net SCL: now reaches U1.9 (GPIO9)
- net SCL: now also J3.2 (Pin_2)
