File: Bimasakti BM-13 EVO/PCB/Wheelspeed Module/Wheelspeed New/Wheelspeed New.kicad_pcb (KiCad board)
At the start: 2 copper layers, 32 x 46.5 mm, 21 parts, among them J3 Conn_01x15_Pin, J4 Conn_01x15_Pin, U1 ESP32-C3_SUPERMINI_TH, U2 LM393

Commit message: tv board FIXXXXX
Parts:
- removed FL, FR, RL, RR: TestPoint, TestPoint:TestPoint_Bridge_Pitch2.54mm_Drill0.7mm
- added TP_FL1: TestPoint, TestPoint:TestPoint_Bridge_Pitch2.54mm_Drill0.7mm, F.Cu at (120.0, 139.0)
- added TP_FR1: TestPoint, TestPoint:TestPoint_Bridge_Pitch2.54mm_Drill0.7mm, F.Cu at (120.0, 136.5)
- added TP_RL1: TestPoint, TestPoint:TestPoint_Bridge_Pitch2.54mm_Drill0.7mm, F.Cu at (120.0, 131.5)
- added TP_RR1: TestPoint, TestPoint:TestPoint_Bridge_Pitch2.54mm_Drill0.7mm, F.Cu at (120.0, 134.0)
Connections:
- J4 pad 10: unconnected-(J4-Pin_10-Pad10) -> /WS_RR_Signal
- J4 pad 11: unconnected-(J4-Pin_11-Pad11) -> /WS_FR_Signal
- J4 pad 12: unconnected-(J4-Pin_12-Pad12) -> /WS_FL_Signal
- J4 pad 9: unconnected-(J4-Pin_9-Pad9) -> /WS_RL_Signal
Routing:
- net /WS_FR_Signal: track 44.0 -> 55.2 mm
- net /WS_RR_Signal: track 36.9 -> 43.8 mm
- net /WS_RL_Signal: track 29.1 -> 36.0 mm
- net /WS_FL_Signal: track 53.4 -> 57.7 mm, vias 0 -> 2

Commit message: kontol tadi ga kesave
Connections:
- J3 pad 1: unconnected-(J3-Pin_1-Pad1) -> /SDA
- J3 pad 2: unconnected-(J3-Pin_2-Pad2) -> /SCL
- J4 pad 3: GND -> unconnected-(J4-Pin_3-Pad3)
- U1 pad 8: unconnected-(U1-GPIO8-Pad8) -> /SDA
- U1 pad 9: unconnected-(U1-GPIO9-Pad9) -> /SCL
Routing:
- net /SCL: track 0.00 -> 10.9 mm
- net /SDA: track 0.00 -> 10.4 mm
Changed lines of the file:
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@@
 	(net 17 "/TX")
 	(net 18 "unconnected-(J4-Pin_14-Pad14)")
-	(net 19 "unconnected-(J3-Pin_1-Pad1)")
-	(net 20 "unconnected-(J3-Pin_2-Pad2)")
-	(net 21 "unconnected-(J4-Pin_8-Pad8)")
-	(net 22 "unconnected-(J4-Pin_6-Pad6)")
-	(net 23 "unconnected-(J4-Pin_2-Pad2)")
-	(net 24 "unconnected-(U1-GPIO4-Pad4)")
-	(net 25 "unconnected-(U1-GPIO7-Pad7)")
-	(net 26 "unconnected-(U1-GPIO8-Pad8)")
-	(net 27 "unconnected-(U1-GPIO5-Pad5)")
-	(net 28 "unconnected-(U1-GPIO6-Pad6)")
-	(net 29 "unconnected-(U1-GPIO10-Pad10)")
-	(net 30 "unconnected-(U1-GPIO9-Pad9)")
+	(net 19 "unconnected-(J4-Pin_8-Pad8)")
+	(net 20 "unconnected-(J4-Pin_6-Pad6)")
+	(net 21 "unconnected-(J4-Pin_2-Pad2)")
+	(net 22 "unconnected-(U1-GPIO4-Pad4)")
+	(net 23 "unconnected-(U1-GPIO7-Pad7)")
+	(net 24 "/SDA")
+	(net 25 "unconnected-(U1-GPIO5-Pad5)")
+	(net 26 "unconnected-(U1-GPIO6-Pad6)")
+	(net 27 "unconnected-(U1-GPIO10-Pad10)")
+	(net 28 "/SCL")
+	(net 29 "unconnected-(J4-Pin_3-Pad3)")
 	(footprint "LM393:SO8_STM"
 		(layer "F.Cu")
@@
 			(size 3.025 1.524)
 			(layers "F.Cu" "F.Mask" "F.Paste")
-			(net 24 "unconnected-(U1-GPIO4-Pad4)")
+			(net 22 "unconnected-(U1-GPIO4-Pad4)")
 			(pinfunction "GPIO4")
 			(pintype "bidirectional")
@@
 			(size 3.025 1.524)
 			(layers "F.Cu" "F.Mask" "F.Paste")
-			(net 27 "unconnected-(U1-GPIO5-Pad5)")
+			(net 25 "unconnected-(U1-GPIO5-Pad5)")
 			(pinfunction "GPIO5")
 			(pintype "bidirectional")
@@
 			(size 3.025 1.524)
 			(layers "F.Cu" "F.Mask" "F.Paste")
-			(net 28 "unconnected-(U1-GPIO6-Pad6)")
+			(net 26 "unconnected-(U1-GPIO6-Pad6)")
 			(pinfunction "GPIO6")
 			(pintype "bidirectional")
@@
 			(size 3.025 1.524)
 			(layers "F.Cu" "F.Mask" "F.Paste")
-			(net 25 "unconnected-(U1-GPIO7-Pad7)")
+			(net 23 "unconnected-(U1-GPIO7-Pad7)")
 			(pinfunction "GPIO7")
 			(pintype "bidirectional")
@@
 			(size 3.025 1.524)
 			(layers "F.Cu" "F.Mask" "F.Paste")
-			(net 26 "unconnected-(U1-GPIO8-Pad8)")
+			(net 24 "/SDA")
 			(pinfunction "GPIO8")
 			(pintype "bidirectional")
@@
 			(size 3.025 1.524)
 			(layers "F.Cu" "F.Mask" "F.Paste")
-			(net 30 "unconnected-(U1-GPIO9-Pad9)")
+			(net 28 "/SCL")
 			(pinfunction "GPIO9")
 			(pintype "bidirectional")
@@
 			(size 3.025 1.524)
 			(layers "F.Cu" "F.Mask" "F.Paste")
-			(net 29 "unconnected-(U1-GPIO10-Pad10)")
+			(net 27 "unconnected-(U1-GPIO10-Pad10)")
 			(pinfunction "GPIO10")
 			(pintype "bidirectional")
@@
 			(layers "*.Cu" "*.Mask")
 			(remove_unused_layers no)
-			(net 23 "unconnected-(J4-Pin_2-Pad2)")
+			(net 21 "unconnected-(J4-Pin_2-Pad2)")
 			(pinfunction "Pin_2")
 			(pintype "passive")
@@
 			(layers "*.Cu" "*.Mask")
 			(remove_unused_layers no)
-			(net 2 "GND")
+			(net 29 "unconnected-(J4-Pin_3-Pad3)")
 			(pinfunction "Pin_3")
 			(pintype "passive")
@@
 			(layers "*.Cu" "*.Mask")
 			(remove_unused_layers no)
-			(net 22 "unconnected-(J4-Pin_6-Pad6)")
+			(net 20 "unconnected-(J4-Pin_6-Pad6)")
 			(pinfunction "Pin_6")
 			(pintype "passive")
@@
 			(layers "*.Cu" "*.Mask")
 			(remove_unused_layers no)
-			(net 21 "unconnected-(J4-Pin_8-Pad8)")
+			(net 19 "unconnected-(J4-Pin_8-Pad8)")
 			(pinfunction "Pin_8")
 			(pintype "passive")
@@
 			(layers "*.Cu" "*.Mask")
 			(remove_unused_layers no)
-			(net 19 "unconnected-(J3-Pin_1-Pad1)")
+			(net 24 "/SDA")
 			(pinfunction "Pin_1")
 			(pintype "passive")
@@
 			(layers "*.Cu" "*.Mask")
 			(remove_unused_layers no)
-			(net 20 "unconnected-(J3-Pin_2-Pad2)")
+			(net 28 "/SCL")
 			(pinfunction "Pin_2")
 			(pintype "passive")
@@
 		(net 17)
 	)
+	(segment
+		(start 104.75 113.1915)
+		(end 104.75 108.75)
+		(width 0.6)
+		(layer "F.Cu")
+		(net 24)
+	)
+	(segment
+		(start 107.015 114.72)
+		(end 106.2785 114.72)
+		(width 0.6)
+		(layer "F.Cu")
+		(net 24)
+	)
+	(segment
+		(start 104.75 108.75)
+		(end 104 108)
+		(width 0.6)
+		(layer "F.Cu")
+		(net 24)
+	)
+	(segment
+		(start 106.2785 114.72)
+		(end 104.75 113.1915)
+		(width 0.6)
+		(layer "F.Cu")
+		(net 24)
+	)
+	(segment
+		(start 104 108)
+		(end 102 108)
+		(width 0.6)
+		(layer "F.Cu")
+		(net 24)
+	)
+	(segment
+		(start 102.79 110.54)
+		(end 103.75 111.5)
+		(width 0.6)
+		(layer "F.Cu")
+		(net 28)
+	)
+	(segment
+		(start 103.75 111.5)
+		(end 103.75 116.75)
+		(width 0.6)
+		(layer "F.Cu")
+		(net 28)
+	)
+	(segment
+		(start 104.26 117.26)
+		(end 107.015 117.26)
+		(width 0.6)
+		(layer "F.Cu")
+		(net 28)
+	)
+	(segment
+		(start 102 110.54)
+		(end 102.79 110.54)
+		(width 0.6)
+		(layer "F.Cu")
+		(net 28)
+	)
+	(segment
+		(start 103.75 116.75)
+		(end 104.26 117.26)
+		(width 0.6)
+		(layer "F.Cu")
+		(net 28)
+	)
 	(zone

Commit message: tambah i2c di tele
Parts:
- renumbered TP_FL1 to FL, TP_FR1 to FR, TP_RL1 to RL, TP_RR1 to RR
Connections:
- J4 pad 2: unconnected-(J4-Pin_2-Pad2) -> GND
- J4 pad 3: unconnected-(J4-Pin_3-Pad3) -> GND
- J4 pad 6: unconnected-(J4-Pin_6-Pad6) -> GND
- J4 pad 8: unconnected-(J4-Pin_8-Pad8) -> GND
Routing:
- net /WS_FR_Signal: track 55.2 -> 55.9 mm
Changed lines of the file:
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@@
 	(net 17 "/TX")
 	(net 18 "unconnected-(J4-Pin_14-Pad14)")
-	(net 19 "unconnected-(J4-Pin_8-Pad8)")
-	(net 20 "unconnected-(J4-Pin_6-Pad6)")
-	(net 21 "unconnected-(J4-Pin_2-Pad2)")
-	(net 22 "unconnected-(U1-GPIO4-Pad4)")
-	(net 23 "unconnected-(U1-GPIO7-Pad7)")
-	(net 24 "/SDA")
-	(net 25 "unconnected-(U1-GPIO5-Pad5)")
-	(net 26 "unconnected-(U1-GPIO6-Pad6)")
-	(net 27 "unconnected-(U1-GPIO10-Pad10)")
-	(net 28 "/SCL")
-	(net 29 "unconnected-(J4-Pin_3-Pad3)")
+	(net 19 "unconnected-(U1-GPIO4-Pad4)")
+	(net 20 "unconnected-(U1-GPIO7-Pad7)")
+	(net 21 "/SDA")
+	(net 22 "unconnected-(U1-GPIO5-Pad5)")
+	(net 23 "unconnected-(U1-GPIO6-Pad6)")
+	(net 24 "unconnected-(U1-GPIO10-Pad10)")
+	(net 25 "/SCL")
 	(footprint "LM393:SO8_STM"
 		(layer "F.Cu")
@@
 		(descr "wire loop as test point, pitch 2.0mm, hole diameter 0.7mm, wire diameter 0.5mm")
 		(tags "test point wire loop")
-		(property "Reference" "TP_FR1"
-			(at 1.1 1.7 0)
+		(property "Reference" "FR"
+			(at -2.21 0 0)
 			(layer "F.SilkS")
 			(effects
@@
 		(descr "wire loop as test point, pitch 2.0mm, hole diameter 0.7mm, wire diameter 0.5mm")
 		(tags "test point wire loop")
-		(property "Reference" "TP_RL1"
-			(at 1.1 1.7 0)
+		(property "Reference" "RL"
+			(at -2.21 0 0)
 			(layer "F.SilkS")
 			(effects
@@
 		(descr "wire loop as test point, pitch 2.0mm, hole diameter 0.7mm, wire diameter 0.5mm")
 		(tags "test point wire loop")
-		(property "Reference" "TP_RR1"
-			(at 1.1 1.7 0)
+		(property "Reference" "RR"
+			(at -2.21 0 0)
 			(layer "F.SilkS")
 			(effects
@@
 		(descr "wire loop as test point, pitch 2.0mm, hole diameter 0.7mm, wire diameter 0.5mm")
 		(tags "test point wire loop")
-		(property "Reference" "TP_FL1"
-			(at 1.1 1.7 0)
+		(property "Reference" "FL"
+			(at -2.21 0 0)
 			(layer "F.SilkS")
 			(effects
@@
 			(size 3.025 1.524)
 			(layers "F.Cu" "F.Mask" "F.Paste")
-			(net 22 "unconnected-(U1-GPIO4-Pad4)")
+			(net 19 "unconnected-(U1-GPIO4-Pad4)")
 			(pinfunction "GPIO4")
 			(pintype "bidirectional")
@@
 			(size 3.025 1.524)
 			(layers "F.Cu" "F.Mask" "F.Paste")
-			(net 25 "unconnected-(U1-GPIO5-Pad5)")
+			(net 22 "unconnected-(U1-GPIO5-Pad5)")
 			(pinfunction "GPIO5")
 			(pintype "bidirectional")
@@
 			(size 3.025 1.524)
 			(layers "F.Cu" "F.Mask" "F.Paste")
-			(net 26 "unconnected-(U1-GPIO6-Pad6)")
+			(net 23 "unconnected-(U1-GPIO6-Pad6)")
 			(pinfunction "GPIO6")
 			(pintype "bidirectional")
@@
 			(size 3.025 1.524)
 			(layers "F.Cu" "F.Mask" "F.Paste")
-			(net 23 "unconnected-(U1-GPIO7-Pad7)")
+			(net 20 "unconnected-(U1-GPIO7-Pad7)")
 			(pinfunction "GPIO7")
 			(pintype "bidirectional")
@@
 			(size 3.025 1.524)
 			(layers "F.Cu" "F.Mask" "F.Paste")
-			(net 24 "/SDA")
+			(net 21 "/SDA")
 			(pinfunction "GPIO8")
 			(pintype "bidirectional")
@@
 			(size 3.025 1.524)
 			(layers "F.Cu" "F.Mask" "F.Paste")
-			(net 28 "/SCL")
+			(net 25 "/SCL")
 			(pinfunction "GPIO9")
 			(pintype "bidirectional")
@@
 			(size 3.025 1.524)
 			(layers "F.Cu" "F.Mask" "F.Paste")
-			(net 27 "unconnected-(U1-GPIO10-Pad10)")
+			(net 24 "unconnected-(U1-GPIO10-Pad10)")
 			(pinfunction "GPIO10")
 			(pintype "bidirectional")
@@
 			(layers "*.Cu" "*.Mask")
 			(remove_unused_layers no)
-			(net 21 "unconnected-(J4-Pin_2-Pad2)")
+			(net 2 "GND")
 			(pinfunction "Pin_2")
 			(pintype "passive")
@@
 			(layers "*.Cu" "*.Mask")
 			(remove_unused_layers no)
-			(net 29 "unconnected-(J4-Pin_3-Pad3)")
+			(net 2 "GND")
 			(pinfunction "Pin_3")
 			(pintype "passive")
@@
 			(layers "*.Cu" "*.Mask")
 			(remove_unused_layers no)
-			(net 20 "unconnected-(J4-Pin_6-Pad6)")
+			(net 2 "GND")
 			(pinfunction "Pin_6")
 			(pintype "passive")
@@
 			(layers "*.Cu" "*.Mask")
 			(remove_unused_layers no)
-			(net 19 "unconnected-(J4-Pin_8-Pad8)")
+			(net 2 "GND")
 			(pinfunction "Pin_8")
 			(pintype "passive")
@@
 			(layers "*.Cu" "*.Mask")
 			(remove_unused_layers no)
-			(net 24 "/SDA")
+			(net 21 "/SDA")
 			(pinfunction "Pin_1")
 			(pintype "passive")
@@
 			(layers "*.Cu" "*.Mask")
 			(remove_unused_layers no)
-			(net 28 "/SCL")
+			(net 25 "/SCL")
 			(pinfunction "Pin_2")
 			(pintype "passive")
@@
 	)
 	(segment
-		(start 123.7 119.8)
-		(end 122.985 119.8)
-		(width 0.4)
-		(layer "F.Cu")
-		(net 6)
-	)
-	(segment
-		(start 120.5 127.5)
-		(end 124.75 127.5)
+		(start 125.399 126.851)
+		(end 125.399 121.499)
 		(width 0.4)
 		(layer "F.Cu")
@@
 	)
 	(segment
-		(start 117.6 136.6)
-		(end 117.6 130.4)
+		(start 125.399 121.499)
+		(end 123.7 119.8)
 		(width 0.4)
 		(layer "F.Cu")
@@
 	)
 	(segment
-		(start 117.6 130.4)
-		(end 120.5 127.5)
+		(start 124.75 127.5)
+		(end 125.399 126.851)
 		(width 0.4)
 		(layer "F.Cu")
@@
 	)
 	(segment
-		(start 124.75 127.5)
-		(end 125.399 126.851)
+		(start 123.7 119.8)
+		(end 122.985 119.8)
 		(width 0.4)
 		(layer "F.Cu")
@@
 	)
 	(segment
-		(start 125.399 126.851)
-		(end 125.399 121.499)
+		(start 117.6 136.6)
+		(end 117.6 129.15)
 		(width 0.4)
 		(layer "F.Cu")
@@
 	)
 	(segment
-		(start 125.399 121.499)
-		(end 123.7 119.8)
-		(width 0.4)
-		(layer "F.Cu")
-		(net 6)
-	)
-	(segment
 		(start 110.40415 134.7)
 		(end 115.2 134.7)
@@
 	)
 	(segment
+		(start 119.25 127.5)
+		(end 124.75 127.5)
+		(width 0.4)
+		(layer "F.Cu")
+		(net 6)
+	)
+	(segment
 		(start 115.2 134.7)
 		(end 117.1 136.6)
@@
 	)
 	(segment
+		(start 117.6 129.15)
+		(end 119.25 127.5)
+		(width 0.4)
+		(layer "F.Cu")
+		(net 6)
+	)
+	(segment
 		(start 118.2 136.6)
 		(end 122.8 136.6)
@@
 	)
 	(segment
-		(start 108.9 142.4)
-		(end 109.6 141.7)
-		(width 0.4)
-		(layer "F.Cu")
-		(net 10)
-	)
-	(segment
-		(start 107.775 144.5875)
-		(end 107.7875 144.6)
+		(start 108.5 142.4)
+		(end 108.9 142.4)
 		(width 0.4)
 		(layer "F.Cu")
@@
 	)
 	(segment
-		(start 107.785 143.115)
-		(end 108.5 142.4)
+		(start 107.785 143.5)
+		(end 107.785 143.115)
 		(width 0.4)
 		(layer "F.Cu")
@@
 	)
 	(segment
-		(start 108.5 142.4)
-		(end 108.9 142.4)
+		(start 107.775 144.5875)
+		(end 107.7875 144.6)
 		(width 0.4)
 		(layer "F.Cu")
@@
 	)
 	(segment
-		(start 107.785 143.5)
-		(end 107.785 143.115)
+		(start 109.6 141.7)
+		(end 109.6 139.6256)
 		(width 0.4)
 		(layer "F.Cu")
@@
 	)
 	(segment
-		(start 109.6 141.7)
-		(end 109.6 139.6256)
+		(start 108.9 142.4)
+		(end 109.6 141.7)
 		(width 0.4)
 		(layer "F.Cu")
@@
 	)
 	(segment
+		(start 107.785 143.115)
+		(end 108.5 142.4)
+		(width 0.4)
+		(layer "F.Cu")
+		(net 10)
+	)
+	(segment
 		(start 108.7394 138.765)
 		(end 108.27585 138.765)
@@
 		(width 0.6)
 		(layer "F.Cu")
-		(net 24)
+		(net 21)
 	)
 	(segment
@@
 		(width 0.6)
 		(layer "F.Cu")
-		(net 24)
+		(net 21)
 	)
 	(segment
@@
 		(width 0.6)
 		(layer "F.Cu")
-		(net 24)
+		(net 21)
 	)
 	(segment
@@
 		(width 0.6)
 		(layer "F.Cu")
-		(net 24)
+		(net 21)
 	)
 	(segment
@@
 		(width 0.6)
 		(layer "F.Cu")
-		(net 24)
+		(net 21)
 	)
 	(segment
@@
 		(width 0.6)
 		(layer "F.Cu")
-		(net 28)
+		(net 25)
 	)
 	(segment
@@
 		(width 0.6)
 		(layer "F.Cu")
-		(net 28)
+		(net 25)
 	)
 	(segment
@@
 		(width 0.6)
 		(layer "F.Cu")
-		(net 28)
+		(net 25)
 	)
 	(segment
@@
 		(width 0.6)
 		(layer "F.Cu")
-		(net 28)
+		(net 25)
 	)
 	(segment
@@
 		(width 0.6)
 		(layer "F.Cu")
-		(net 28)
+		(net 25)
 	)
 	(zone
