File: Bimasakti BM-13 EVO/PCB/Telemetry/Telemetry V.3 BM13 EVO Hy.kicad_pcb (KiCad board)
At the start: 2 copper layers, 83.5 x 70 mm, 28 parts, among them J1 MSD-4-A, J2 CON INT/32, J4 Conn_01x16_Pin, U1 ESP32-DEVKIT-V1, U2 74LVC125APW_118, U3 DS3231SN_

Commit message: tambah i2c di tele
Connections:
- J4 pad 15: GND -> /SDA
- J4 pad 16: GND -> /SCL
Routing:
- net /SDA: track 19.9 -> 65.9 mm
- net /SCL: track 34.3 -> 71.8 mm
Changed lines of the file:
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@@
 			(layer "F.Fab")
 		)
-		(pad "" np_thru_hole circle
-			(at -12.28 -23.475 180)
-			(size 3 3)
-			(drill 3)
-			(layers "*.Cu" "*.Mask")
-		)
-		(pad "" np_thru_hole circle
-			(at -12.28 23.475 180)
-			(size 3 3)
-			(drill 3)
-			(layers "*.Cu" "*.Mask")
-		)
-		(pad "" np_thru_hole circle
-			(at 12.23 -23.475 180)
-			(size 3 3)
-			(drill 3)
-			(layers "*.Cu" "*.Mask")
-		)
-		(pad "" np_thru_hole circle
-			(at 12.23 23.475 180)
-			(size 3 3)
-			(drill 3)
-			(layers "*.Cu" "*.Mask")
-		)
 		(pad "1" thru_hole rect
 			(at -12.7 -15.515 180)
@@
 			(solder_mask_margin 0.102)
 		)
-		(zone
-			(net 0)
-			(net_name "")
-			(layer "F.Cu")
-			(hatch full 0.508)
-			(connect_pads
-				(clearance 0)
-			)
-			(min_thickness 0.01)
-			(filled_areas_thickness no)
-			(keepout
-				(tracks not_allowed)
-				(vias not_allowed)
-				(pads not_allowed)
-				(copperpour not_allowed)
-				(footprints allowed)
-			)
-			(placement
-				(enabled no)
-				(sheetname "")
-			)
-			(fill
-				(thermal_gap 0.508)
-				(thermal_bridge_width 0.508)
-			)
-			(polygon
-				(pts
-					(xy 84.41 60.765) (xy 66.72 60.765) (xy 66.72 54.275) (xy 84.41 54.275)
-				)
-			)
-		)
-		(zone
-			(net 0)
-			(net_name "")
-			(layers "F.Cu" "B.Cu")
-			(hatch full 0.508)
-			(connect_pads
-				(clearance 0)
-			)
-			(min_thickness 0.01)
-			(filled_areas_thickness no)
-			(keepout
-				(tracks allowed)
-				(vias not_allowed)
-				(pads allowed)
-				(copperpour allowed)
-				(footprints allowed)
-			)
-			(placement
-				(enabled no)
-				(sheetname "")
-			)
-			(fill
-				(thermal_gap 0.508)
-				(thermal_bridge_width 0.508)
-			)
-			(polygon
-				(pts
-					(xy 84.41 60.765) (xy 66.72 60.765) (xy 66.72 54.275) (xy 84.41 54.275)
-				)
-			)
-		)
-		(zone
-			(net 0)
-			(net_name "")
-			(layer "B.Cu")
-			(hatch full 0.508)
-			(connect_pads
-				(clearance 0)
-			)
-			(min_thickness 0.01)
-			(filled_areas_thickness no)
-			(keepout
-				(tracks not_allowed)
-				(vias not_allowed)
-				(pads not_allowed)
-				(copperpour not_allowed)
-				(footprints allowed)
-			)
-			(placement
-				(enabled no)
-				(sheetname "")
-			)
-			(fill
-				(thermal_gap 0.508)
-				(thermal_bridge_width 0.508)
-			)
-			(polygon
-				(pts
-					(xy 84.41 60.765) (xy 66.72 60.765) (xy 66.72 54.275) (xy 84.41 54.275)
-				)
-			)
-		)
 		(embedded_fonts no)
 		(model "D:/Arjunda/Library/kicad/ESP32/ESP32_DevKitV1.step"
@@
 			(layers "*.Cu" "*.Mask")
 			(remove_unused_layers no)
-			(net 1 "GND")
+			(net 25 "/SDA")
 			(pinfunction "Pin_15")
 			(pintype "passive")
@@
 			(layers "*.Cu" "*.Mask")
 			(remove_unused_layers no)
-			(net 1 "GND")
+			(net 26 "/SCL")
 			(pinfunction "Pin_16")
 			(pintype "passive")
@@
 	)
 	(segment
+		(start 59.25 59.5)
+		(end 61.25 57.5)
+		(width 0.5)
+		(layer "B.Cu")
+		(net 25)
+	)
+	(segment
+		(start 61.25 57.5)
+		(end 76.75 57.5)
+		(width 0.5)
+		(layer "B.Cu")
+		(net 25)
+	)
+	(segment
+		(start 79.5 68)
+		(end 81.365 69.865)
+		(width 0.5)
+		(layer "B.Cu")
+		(net 25)
+	)
+	(segment
+		(start 58.31 64.44)
+		(end 59.25 63.5)
+		(width 0.5)
+		(layer "B.Cu")
+		(net 25)
+	)
+	(segment
+		(start 81.365 69.865)
+		(end 88.2 69.865)
+		(width 0.5)
+		(layer "B.Cu")
+		(net 25)
+	)
+	(segment
+		(start 76.75 57.5)
+		(end 79.5 60.25)
+		(width 0.5)
+		(layer "B.Cu")
+		(net 25)
+	)
+	(segment
+		(start 57 64.44)
+		(end 58.31 64.44)
+		(width 0.5)
+		(layer "B.Cu")
+		(net 25)
+	)
+	(segment
+		(start 59.25 63.5)
+		(end 59.25 59.5)
+		(width 0.5)
+		(layer "B.Cu")
+		(net 25)
+	)
+	(segment
+		(start 79.5 60.25)
+		(end 79.5 68)
+		(width 0.5)
+		(layer "B.Cu")
+		(net 25)
+	)
+	(segment
 		(start 106 64.6)
 		(end 104.2 62.8)
@@
 		(net 26)
 	)
+	(segment
+		(start 57 59.75)
+		(end 57 61.9)
+		(width 0.4)
+		(layer "B.Cu")
+		(net 26)
+	)
+	(segment
+		(start 60.75 56)
+		(end 57 59.75)
+		(width 0.4)
+		(layer "B.Cu")
+		(net 26)
+	)
+	(segment
+		(start 84.995 62.245)
+		(end 78.75 56)
+		(width 0.4)
+		(layer "B.Cu")
+		(net 26)
+	)
+	(segment
+		(start 78.75 56)
+		(end 60.75 56)
+		(width 0.4)
+		(layer "B.Cu")
+		(net 26)
+	)
+	(segment
+		(start 88.2 62.245)
+		(end 84.995 62.245)
+		(width 0.4)
+		(layer "B.Cu")
+		(net 26)
+	)
