File: Bimasakti BM-13 EVO/PCB/Telemetry/Telemetry V.3 BM13 EVO Hy.kicad_sch (KiCad schematic)
At the start: 23 parts, among them J1 MSD-4-A, J2 CON INT/32, J4 Conn_01x04_Socket, U1 ESP32-DEVKIT-V1, U2 74LVC125APW_118, U3 DS3231SN_

Commit message: Telemetry Finish
Parts:
- removed J4: Conn_01x04_Socket, Connector_JST:JST_XH_B4B-XH-A_1x04_P2.50mm_Vertical, symbol Connector:Conn_01x04_Socket
- added J4: Conn_01x16_Pin, Connector_PinHeader_2.54mm:PinHeader_1x16_P2.54mm_Vertical, symbol Connector:Conn_01x16_Pin
Connections:
- net +5V: now also J4.6 (Pin_6)
- net GND: now also J4.11 (Pin_11)
- net LED1: now also U1.4 (D2); no longer U1.20 (D35)
- net LED2: now also U1.5 (D4); no longer U1.19 (D34)
- net SCK2: now reaches U1.26 (D14)
- net SCK2: now also J4.9 (Pin_9)
- net MISO2: now reaches U1.27 (D12)
- net MISO2: now also J4.8 (Pin_8)
- net MOSI2: now reaches U1.28 (D13)
- net MOSI2: now also J4.7 (Pin_7)
- net CS2: now reaches U1.3 (D15)
- net CS2: now also J4.10 (Pin_10)

Commit message: Aku Telemetry
Connections:
- net GND: now also J4.1 (Pin_1), J4.12 (Pin_12), J4.13 (Pin_13), J4.14 (Pin_14), J4.15 (Pin_15), J4.16 (Pin_16), J4.2 (Pin_2), J4.3 (Pin_3), J4.4 (Pin_4), J4.5 (Pin_5)
Other:
- moved on the sheet: D3, J4, R7

Commit message: Asu
Connections:
- net +5V: now also J4.1 (Pin_1); no longer J4.6 (Pin_6)
- net CS2: now also J4.5 (Pin_5); no longer J4.10 (Pin_10)
- net GND: now also J4.10 (Pin_10), J4.9 (Pin_9); no longer J4.1 (Pin_1), J4.5 (Pin_5)
- net MISO2: now also J4.7 (Pin_7); no longer J4.8 (Pin_8)
- net MOSI2: now also J4.6 (Pin_6); no longer J4.7 (Pin_7)
- net SCK2: now also J4.8 (Pin_8); no longer J4.9 (Pin_9)
Changed lines of the file:
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@@
 	(wire
 		(pts
-			(xy 254 140.97) (xy 262.89 140.97)
+			(xy 130.81 110.49) (xy 135.89 110.49)
 		)
 		(stroke
@@
 	(wire
 		(pts
-			(xy 130.81 125.73) (xy 137.16 125.73)
+			(xy 254 140.97) (xy 262.89 140.97)
 		)
 		(stroke
@@
 	(wire
 		(pts
-			(xy 139.7 177.8) (xy 143.51 177.8)
+			(xy 130.81 125.73) (xy 137.16 125.73)
 		)
 		(stroke
@@
 	(wire
 		(pts
-			(xy 130.81 120.65) (xy 135.89 120.65)
+			(xy 139.7 177.8) (xy 143.51 177.8)
 		)
 		(stroke
@@
 	(wire
 		(pts
-			(xy 130.81 92.71) (xy 135.89 92.71)
+			(xy 196.85 144.78) (xy 193.04 144.78)
 		)
 		(stroke
@@
 	(wire
 		(pts
-			(xy 196.85 144.78) (xy 193.04 144.78)
+			(xy 130.81 44.45) (xy 138.43 44.45)
 		)
 		(stroke
@@
 	(wire
 		(pts
-			(xy 130.81 44.45) (xy 138.43 44.45)
+			(xy 130.81 107.95) (xy 135.89 107.95)
 		)
 		(stroke
@@
 	(wire
 		(pts
+			(xy 130.81 120.65) (xy 135.89 120.65)
+		)
+		(stroke
+			(width 0)
+			(type default)
+		)
+	)
+	(wire
+		(pts
+			(xy 130.81 102.87) (xy 135.89 102.87)
+		)
+		(stroke
+			(width 0)
+			(type default)
+		)
+	)
+	(wire
+		(pts
 			(xy 161.29 93.98) (xy 162.56 93.98)
 		)
@@
 	(wire
 		(pts
-			(xy 130.81 115.57) (xy 135.89 115.57)
+			(xy 224.79 31.75) (xy 232.41 31.75)
 		)
 		(stroke
@@
 	(wire
 		(pts
-			(xy 224.79 31.75) (xy 232.41 31.75)
+			(xy 130.81 115.57) (xy 135.89 115.57)
 		)
 		(stroke
@@
 	(wire
 		(pts
-			(xy 237.49 95.25) (xy 237.49 97.79)
+			(xy 130.81 118.11) (xy 135.89 118.11)
 		)
 		(stroke
@@
 	(wire
 		(pts
-			(xy 193.04 31.75) (xy 193.04 35.56)
+			(xy 237.49 95.25) (xy 237.49 97.79)
 		)
 		(stroke
@@
 	(wire
 		(pts
-			(xy 158.75 127) (xy 162.56 127)
+			(xy 193.04 31.75) (xy 193.04 35.56)
 		)
 		(stroke
@@
 	(wire
 		(pts
-			(xy 254 143.51) (xy 254 140.97)
+			(xy 158.75 127) (xy 162.56 127)
 		)
 		(stroke
@@
 	(wire
 		(pts
-			(xy 231.14 67.31) (xy 231.14 69.85)
+			(xy 254 143.51) (xy 254 140.97)
 		)
 		(stroke
@@
 	(wire
 		(pts
-			(xy 130.81 105.41) (xy 135.89 105.41)
+			(xy 231.14 67.31) (xy 231.14 69.85)
 		)
 		(stroke
@@
 	(wire
 		(pts
-			(xy 130.81 118.11) (xy 135.89 118.11)
-		)
-		(stroke
-			(width 0)
-			(type default)
-		)
-	)
-	(wire
-		(pts
 			(xy 254 133.35) (xy 262.89 133.35)
 		)
@@
 	(wire
 		(pts
-			(xy 130.81 107.95) (xy 135.89 107.95)
-		)
-		(stroke
-			(width 0)
-			(type default)
-		)
-	)
-	(wire
-		(pts
 			(xy 231.14 54.61) (xy 241.3 54.61)
 		)
@@
 	(wire
 		(pts
-			(xy 130.81 102.87) (xy 135.89 102.87)
-		)
-		(stroke
-			(width 0)
-			(type default)
-		)
-	)
-	(wire
-		(pts
 			(xy 130.81 46.99) (xy 147.32 46.99)
 		)
@@
 	(wire
 		(pts
-			(xy 130.81 110.49) (xy 135.89 110.49)
+			(xy 130.81 97.79) (xy 135.89 97.79)
 		)
 		(stroke
@@
 	(wire
 		(pts
-			(xy 130.81 97.79) (xy 135.89 97.79)
+			(xy 251.46 140.97) (xy 254 140.97)
 		)
 		(stroke
@@
 	(wire
 		(pts
-			(xy 251.46 140.97) (xy 254 140.97)
+			(xy 237.49 105.41) (xy 237.49 107.95)
 		)
 		(stroke
@@
 	(wire
 		(pts
-			(xy 237.49 105.41) (xy 237.49 107.95)
+			(xy 144.78 49.53) (xy 147.32 49.53)
 		)
 		(stroke
@@
 	(wire
 		(pts
-			(xy 144.78 49.53) (xy 147.32 49.53)
+			(xy 130.81 52.07) (xy 138.43 52.07)
 		)
 		(stroke
@@
 	(wire
 		(pts
-			(xy 130.81 52.07) (xy 138.43 52.07)
+			(xy 130.81 113.03) (xy 135.89 113.03)
 		)
 		(stroke
@@
 	(wire
 		(pts
+			(xy 130.81 105.41) (xy 135.89 105.41)
+		)
+		(stroke
+			(width 0)
+			(type default)
+		)
+	)
+	(wire
+		(pts
 			(xy 139.7 172.72) (xy 143.51 172.72)
 		)
@@
 	(wire
 		(pts
-			(xy 130.81 113.03) (xy 135.89 113.03)
+			(xy 251.46 128.27) (xy 256.54 128.27)
 		)
 		(stroke
@@
 	(wire
 		(pts
-			(xy 251.46 128.27) (xy 256.54 128.27)
+			(xy 130.81 54.61) (xy 147.32 54.61)
 		)
 		(stroke
@@
 	(wire
 		(pts
-			(xy 130.81 54.61) (xy 147.32 54.61)
+			(xy 139.7 166.37) (xy 139.7 167.64)
 		)
 		(stroke
@@
 	(wire
 		(pts
-			(xy 139.7 166.37) (xy 139.7 167.64)
+			(xy 193.04 93.98) (xy 194.31 93.98)
 		)
 		(stroke
@@
 	(wire
 		(pts
-			(xy 193.04 93.98) (xy 194.31 93.98)
+			(xy 139.7 180.34) (xy 143.51 180.34)
 		)
 		(stroke
@@
 	(wire
 		(pts
-			(xy 139.7 180.34) (xy 143.51 180.34)
+			(xy 130.81 92.71) (xy 135.89 92.71)
 		)
 		(stroke
@@
 		)
 	)
+	(label "CS2"
+		(at 135.89 102.87 0)
+		(effects
+			(font
+				(size 1.27 1.27)
+			)
+			(justify left bottom)
+		)
+	)
 	(label "LED1"
 		(at 158.75 116.84 0)
@@
 	)
 	(label "MOSI2"
-		(at 135.89 107.95 0)
+		(at 135.89 105.41 0)
 		(effects
 			(font
@@
 	)
 	(label "SCK2"
-		(at 135.89 113.03 0)
+		(at 135.89 110.49 0)
 		(effects
 			(font
@@
 	)
 	(label "MISO2"
-		(at 135.89 110.49 0)
+		(at 135.89 107.95 0)
 		(effects
 			(font
@@
 		)
 	)
-	(label "CS2"
-		(at 135.89 115.57 0)
-		(effects
-			(font
-				(size 1.27 1.27)
-			)
-			(justify left bottom)
-		)
-	)
 	(label "DO_LLS"
 		(at 204.47 46.99 0)
@@
 		)
 		(property "Value" "GND"
-			(at 137.922 100.076 90)
+			(at 138.176 99.314 90)
 			(effects
 				(font
@@
 	(symbol
 		(lib_id "power:GND")
-		(at 135.89 102.87 90)
+		(at 135.89 113.03 90)
 		(unit 1)
 		(exclude_from_sim no)
@@
 		(dnp no)
 		(property "Reference" "#PWR029"
-			(at 142.24 102.87 0)
+			(at 142.24 113.03 0)
 			(effects
 				(font
@@
 		)
 		(property "Value" "GND"
-			(at 137.922 105.156 90)
+			(at 137.922 115.316 90)
 			(effects
 				(font
@@
 		)
 		(property "Footprint" ""
-			(at 135.89 102.87 0)
+			(at 135.89 113.03 0)
 			(effects
 				(font
@@
 		)
 		(property "Datasheet" ""
-			(at 135.89 102.87 0)
+			(at 135.89 113.03 0)
 			(effects
 				(font
@@
 		)
 		(property "Description" "Power symbol creates a global label with name \"GND\" , ground"
-			(at 135.89 102.87 0)
+			(at 135.89 113.03 0)
 			(effects
 				(font
@@
 	(symbol
 		(lib_id "power:+5V")
-		(at 135.89 105.41 270)
+		(at 135.89 92.71 270)
 		(unit 1)
 		(exclude_from_sim no)
@@
 		(dnp no)
 		(property "Reference" "#PWR025"
-			(at 132.08 105.41 0)
+			(at 132.08 92.71 0)
 			(effects
 				(font
@@
 		)
 		(property "Value" "+5V"
-			(at 138.43 103.124 90)
+			(at 137.922 91.948 90)
 			(effects
 				(font
@@
 		)
 		(property "Footprint" ""
-			(at 135.89 105.41 0)
+			(at 135.89 92.71 0)
 			(effects
 				(font
@@
 		)
 		(property "Datasheet" ""
-			(at 135.89 105.41 0)
+			(at 135.89 92.71 0)
 			(effects
 				(font
@@
 		)
 		(property "Description" "Power symbol creates a global label with name \"+5V\""
-			(at 135.89 105.41 0)
+			(at 135.89 92.71 0)
 			(effects
 				(font
@@
 		)
 		(property "Value" "GND"
-			(at 137.922 102.616 90)
+			(at 138.176 101.346 90)
 			(effects
 				(font
@@
 	(symbol
 		(lib_id "power:GND")
-		(at 135.89 92.71 90)
+		(at 135.89 115.57 90)
 		(unit 1)
 		(exclude_from_sim no)
@@
 		(dnp no)
 		(property "Reference" "#PWR034"
-			(at 142.24 92.71 0)
+			(at 142.24 115.57 0)
 			(effects
 				(font
@@
 		)
 		(property "Value" "GND"
-			(at 137.922 94.996 90)
+			(at 137.922 117.856 90)
 			(effects
 				(font
@@
 		)
 		(property "Footprint" ""
-			(at 135.89 92.71 0)
+			(at 135.89 115.57 0)
 			(effects
 				(font
@@
 		)
 		(property "Datasheet" ""
-			(at 135.89 92.71 0)
+			(at 135.89 115.57 0)
 			(effects
 				(font
@@
 		)
 		(property "Description" "Power symbol creates a global label with name \"GND\" , ground"
-			(at 135.89 92.71 0)
+			(at 135.89 115.57 0)
 			(effects
 				(font

Commit message: tambah i2c di tele
Connections:
- net GND: no longer J4.15 (Pin_15), J4.16 (Pin_16)
- net SCL: now also J4.16 (Pin_16)
- net SDA: now also J4.15 (Pin_15)
Changed lines of the file:
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@@
 	(wire
 		(pts
-			(xy 130.81 130.81) (xy 135.89 130.81)
+			(xy 130.81 130.81) (xy 137.16 130.81)
 		)
 		(stroke
@@
 	(wire
 		(pts
-			(xy 130.81 128.27) (xy 135.89 128.27)
+			(xy 130.81 128.27) (xy 137.16 128.27)
 		)
 		(stroke
@@
 		)
 	)
+	(label "SCL"
+		(at 137.16 130.81 0)
+		(effects
+			(font
+				(size 1.27 1.27)
+			)
+			(justify left bottom)
+		)
+	)
 	(label "MOSI2"
 		(at 158.75 127 0)
@@
 	(label "TX"
 		(at 139.7 172.72 0)
+		(effects
+			(font
+				(size 1.27 1.27)
+			)
+			(justify left bottom)
+		)
+	)
+	(label "SDA"
+		(at 137.16 128.27 0)
 		(effects
 			(font
@@
 	)
 	(symbol
-		(lib_id "power:GND")
-		(at 135.89 130.81 90)
-		(unit 1)
-		(exclude_from_sim no)
-		(in_bom yes)
-		(on_board yes)
-		(dnp no)
-		(property "Reference" "#PWR032"
-			(at 142.24 130.81 0)
-			(effects
-				(font
-					(size 1.27 1.27)
-				)
-				(hide yes)
-			)
-		)
-		(property "Value" "GND"
-			(at 137.922 133.096 90)
-			(effects
-				(font
-					(size 1.27 1.27)
-				)
-				(justify right)
-			)
-		)
-		(property "Footprint" ""
-			(at 135.89 130.81 0)
-			(effects
-				(font
-					(size 1.27 1.27)
-				)
-				(hide yes)
-			)
-		)
-		(property "Datasheet" ""
-			(at 135.89 130.81 0)
-			(effects
-				(font
-					(size 1.27 1.27)
-				)
-				(hide yes)
-			)
-		)
-		(property "Description" "Power symbol creates a global label with name \"GND\" , ground"
-			(at 135.89 130.81 0)
-			(effects
-				(font
-					(size 1.27 1.27)
-				)
-				(hide yes)
-			)
-		)
-		(pin "1"
-		)
-		(instances
-			(project "Telemetry V.3 BM13 EVO Hy"
-				(path "/fbeb1601-7635-4f9f-9982-28a91a051811"
-					(reference "#PWR032")
-					(unit 1)
-				)
-			)
-		)
-	)
-	(symbol
 		(lib_id "Device:R_Small_US")
 		(at 198.12 46.99 90)
@@
 				)
 				(justify right)
+				(hide yes)
 			)
 		)
@@
 					(unit 1)
 				)
-			)
-		)
-	)
-	(symbol
-		(lib_id "power:GND")
-		(at 135.89 128.27 90)
-		(unit 1)
-		(exclude_from_sim no)
-		(in_bom yes)
-		(on_board yes)
-		(dnp no)
-		(property "Reference" "#PWR028"
-			(at 142.24 128.27 0)
-			(effects
-				(font
-					(size 1.27 1.27)
-				)
-				(hide yes)
-			)
-		)
-		(property "Value" "GND"
-			(at 137.922 130.556 90)
-			(effects
-				(font
-					(size 1.27 1.27)
-				)
-				(justify right)
-			)
-		)
-		(property "Footprint" ""
-			(at 135.89 128.27 0)
-			(effects
-				(font
-					(size 1.27 1.27)
-				)
-				(hide yes)
-			)
-		)
-		(property "Datasheet" ""
-			(at 135.89 128.27 0)
-			(effects
-				(font
-					(size 1.27 1.27)
-				)
-				(hide yes)
-			)
-		)
-		(property "Description" "Power symbol creates a global label with name \"GND\" , ground"
-			(at 135.89 128.27 0)
-			(effects
-				(font
-					(size 1.27 1.27)
-				)
-				(hide yes)
-			)
-		)
-		(pin "1"
-		)
-		(instances
-			(project "Telemetry V.3 BM13 EVO Hy"
-				(path "/fbeb1601-7635-4f9f-9982-28a91a051811"
-					(reference "#PWR028")
-					(unit 1)
-				)
