File: Bimasakti BM-13 EVO/PCB/MotherBoard Rev2/Motherboard Newww/VCU.kicad_pcb (KiCad board)
At the start: 2 copper layers, 184 x 205 mm, 35 parts, among them J1 6437288-3, J10 power, J11 6437288-3, J8 SIGNAL 1, J9 SIGNAL 2

Commit message: tambah i2c di tele
Routing:
- net 5V_T: track 211.6 -> 217.0 mm
- net 5V_P: track 220.7 -> 223.0 mm

Commit message: SELESAI MOTHERBOARD NEW
Parts:
- removed 12V: 12V, Connector_JST:JST_XH_B2B-XH-A_1x02_P2.50mm_Vertical
- removed 5V: 5V_5, Connector_JST:JST_XH_B2B-XH-A_1x02_P2.50mm_Vertical
- removed BSPD: 5V_2, Connector_JST:JST_XH_B2B-XH-A_1x02_P2.50mm_Vertical
- removed R2: R, Resistor_SMD:R_0603_1608Metric_Pad0.98x0.95mm_HandSolder
- removed REF** (x4): MountingHole_3.2mm_M3_Pad_Via, MountingHole:MountingHole_3.2mm_M3_Pad_Via
- removed Tele/Pneu: 5V_1, Connector_JST:JST_XH_B2B-XH-A_1x02_P2.50mm_Vertical
- removed VCU: 5V_3, Connector_JST:JST_XH_B2B-XH-A_1x02_P2.50mm_Vertical
- added 12V1: 12V, Connector_JST:JST_XH_B2B-XH-A_1x02_P2.50mm_Vertical, F.Cu at (175.8, 126.8)
- added ALL1: 5V_5, Connector_JST:JST_XH_B2B-XH-A_1x02_P2.50mm_Vertical, F.Cu at (175.8, 148.0)
- added BSPD2: 5V_2, Connector_JST:JST_XH_B2B-XH-A_1x02_P2.50mm_Vertical, F.Cu at (175.8, 157.0)
- added TELEMETRY1: 5V_1, Connector_JST:JST_XH_B2B-XH-A_1x02_P2.50mm_Vertical, F.Cu at (176.0, 166.0)
- added VCU1: 5V_3, Connector_JST:JST_XH_B2B-XH-A_1x02_P2.50mm_Vertical, F.Cu at (175.8, 175.0)
- moved 3V3 0.25 mm to (175.8, 137.2)
Connections:
- J1 pad 1: ESC1_HI -> ESC1_LO
- J1 pad 18: WS_FR -> WS_RL
- J1 pad 2: ESC1_LO -> ESC1_HI
- J1 pad 26: WS_FL -> WS_RR
- J1 pad 27: WS_RR -> WS_FL
- J1 pad 28: WS_RL -> WS_FR
- J1 pad 4: APPS_IN1 -> STEER_IN
- J1 pad 6: STEER_IN -> APPS_IN1
- J1 pad 8: ESC2_HI -> ESC2_LO
- J1 pad 9: ESC2_LO -> ESC2_HI
- J11 pad 32: unconnected-(J11-Pad32) -> GND
- J11 pad 33: unconnected-(J11-Pad33) -> GND
- J8 pad 1: SCK -> STM_RX
- J8 pad 10: STEER_IN -> ESC1_HI
- J8 pad 11: APPS_IN2 -> ESC1_LO
- J8 pad 12: APPS_IN1 -> GND
- J8 pad 2: MISO -> STM_TX
- J8 pad 3: MOSI -> SS
- J8 pad 4: SS -> MOSI
- J8 pad 5: STM_TX -> MISO
- J8 pad 6: STM_RX -> SCK
- J8 pad 7: GND -> APPS_IN1
- J8 pad 8: ESC1_LO -> APPS_IN2
- J8 pad 9: ESC1_HI -> STEER_IN
- J9 pad 10: ESC2_LO -> unconnected-(J9-Pin_10-Pad10)
- J9 pad 11: ESC2_HI -> unconnected-(J9-Pin_11-Pad11)
- J9 pad 2: WS_RL -> WS_FR
- J9 pad 3: WS_RR -> WS_FL
- J9 pad 4: WS_FL -> WS_RR
- J9 pad 5: WS_FR -> WS_RL
- J9 pad 8: unconnected-(J9-Pin_8-Pad8) -> ESC2_HI
- J9 pad 9: unconnected-(J9-Pin_9-Pad9) -> ESC2_LO
- U2 pad 30: GND -> /SDA
- U2 pad 31: GND -> /SCL
- U4 pad 15: GND -> /SDA
- U4 pad 16: GND -> /SCL
Routing:
- net /SDA: track 0.00 -> 130.8 mm
- net /SCL: track 0.00 -> 130.5 mm
- net WS_RL: track 96.4 -> 69.5 mm
- net WS_FR: track 69.5 -> 96.4 mm
- net APPS_IN1: track 39.2 -> 57.4 mm
- net STM_RX: track 109.4 -> 94.6 mm
- net WS_RR: track 86.8 -> 74.8 mm
- net WS_FL: track 74.8 -> 86.8 mm
- net APPS_IN2: track 42.9 -> 54.0 mm
- net ESC1_LO: track 51.7 -> 47.8 mm
- net ESC1_HI: track 51.6 -> 48.0 mm
- net STM_TX: track 108.4 -> 104.9 mm
- net ESC2_HI: track 75.0 -> 78.1 mm
- net STEER_IN: track 46.7 -> 49.1 mm
- net ESC2_LO: track 76.1 -> 77.7 mm
Other:
- board text added: "CONN D Pneu"
- board text added: "STR"
- board text removed: "CONN B Pneu"
- board text removed: "SR"
