File: Bimasakti BM-13 EVO/PCB/MotherBoard Rev2/Motherboard Newww/VCU.kicad_sch (KiCad schematic)
At the start: 26 parts, among them J1 6437288-3, J10 power, J11 6437288-3, J2 12V, J3 3V3_1, J4 5V_5, J5 5V_1, J6 5V_2, J7 5V_3, J8 SIGNAL 1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

Commit message: SELESAI MOTHERBOARD NEW
Parts:
- renumbered J2 to 12V1, J3 to 3V3, J4 to ALL1, J6 to BSPD2, J5 to TELEMETRY1, J7 to VCU1
Connections:
- net APPS_IN1: now also J1.6, J8.7 (Pin_7); no longer J1.4, J8.12 (Pin_12)
- net APPS_IN2: now also J8.8 (Pin_8); no longer J8.11 (Pin_11)
- net ESC1_HI: now also J1.2, J8.10 (Pin_10); no longer J1.1, J8.9 (Pin_9)
- net ESC1_LO: now also J1.1, J8.11 (Pin_11); no longer J1.2, J8.8 (Pin_8)
- net ESC2_HI: now also J1.9, J9.8 (Pin_8); no longer J1.8, J9.11 (Pin_11)
- net ESC2_LO: now also J1.8, J9.9 (Pin_9); no longer J1.9, J9.10 (Pin_10)
- net GND: now also J8.12 (Pin_12); no longer J8.7 (Pin_7), U2.30 (GND), U2.31 (GND), U4.15 (GND), U4.16 (GND)
- net MISO: now also J8.5 (Pin_5); no longer J8.2 (Pin_2)
- net MOSI: now also J8.4 (Pin_4); no longer J8.3 (Pin_3)
- net SCK: now also J8.6 (Pin_6); no longer J8.1 (Pin_1)
- net SS: now also J8.3 (Pin_3); no longer J8.4 (Pin_4)
- net STEER_IN: now also J1.4, J8.9 (Pin_9); no longer J1.6, J8.10 (Pin_10)
- net STM_RX: now also J8.1 (Pin_1); no longer J8.6 (Pin_6)
- net STM_TX: now also J8.2 (Pin_2); no longer J8.5 (Pin_5)
- net WS_FL: now also J1.27, J9.3 (Pin_3); no longer J1.26, J9.4 (Pin_4)
- net WS_FR: now also J1.28, J9.2 (Pin_2); no longer J1.18, J9.5 (Pin_5)
- net WS_RL: now also J1.18, J9.5 (Pin_5); no longer J1.28, J9.2 (Pin_2)
- net WS_RR: now also J1.26, J9.4 (Pin_4); no longer J1.27, J9.3 (Pin_3)
- new net SCL: U2.31 (GND), U4.16 (GND)
- new net SDA: U2.30 (GND), U4.15 (GND)
Other:
- moved on the sheet: J8
