File: Bimasakti BM-13 EVO/PCB/1. Motherboard Rev3/VCU.kicad_sch (KiCad schematic)
At the start: 26 parts, among them J1 6437288-3, J10 power, J11 6437288-3, J8 SIGNAL 1, J9 SIGNAL 2

Commit message: rapiin
Connections:
- net 5V_B: now also TELEMETRY1.1 (Pin_1); no longer BSPD2.1 (Pin_1)
- net 5V_T: now also BSPD2.1 (Pin_1); no longer TELEMETRY1.1 (Pin_1)
