File: Bimasakti BM-13 EVO/PCB/3. Power Delivery management/PDM Motherboard/PDM MOTHERBOARD.kicad_pcb (KiCad board)
At the start: 2 copper layers, 77 x 73.1 mm, 43 parts

Commit message: rapiin
Other:
- board text added: "5V"
Changed lines of the file:
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@@
 	)
 	(gr_line
-		(start 120.43712 35.147151)
+		(start 120.5 35)
 		(end 121.323303 33.528)
 		(stroke
@@
 	)
 	(gr_line
+		(start 120.520558 45.255139)
+		(end 121.343861 43.783139)
+		(stroke
+			(width 0.1)
+			(type default)
+		)
+		(layer "F.SilkS")
+	)
+	(gr_line
 		(start 147.32 57.635917)
 		(end 145.288 57.635917)
@@
 	)
 	(gr_line
-		(start 117.608882 35.147151)
-		(end 120.43712 35.147151)
+		(start 117.608882 35)
+		(end 120.5 35)
 		(stroke
 			(width 0.1)
@@
 		)
 		(fill no)
+		(layer "F.SilkS")
+	)
+	(gr_line
+		(start 117.62944 45.255139)
+		(end 120.520558 45.255139)
+		(stroke
+			(width 0.1)
+			(type default)
+		)
 		(layer "F.SilkS")
 	)
@@
 		)
 	)
+	(gr_text "5V"
+		(at 118.25 45.132463 0)
+		(layer "F.SilkS")
+		(effects
+			(font
+				(size 1 1)
+				(thickness 0.15)
+			)
+			(justify left bottom)
+		)
+	)
 	(gr_text "GND\n"
 		(at 147.052805 75.442855 90)
@@
 	)
 	(gr_text "3V3\n"
-		(at 117.637187 35.052 0)
-		(layer "F.SilkS")
-		(effects
+		(at 117.638636 34.877324 0)
+		(layer "F.SilkS")
+		(effects

Commit message: awawawaaw jlc
Parts:
- added G***: LOGO, LOGO, F.Cu at (101.5, 41.5)
