File: Bimasakti BM-13 EVO/PCB/4. Torque Vectoring Board/Torque Vectoring Board.kicad_pcb (KiCad board)
At the start: 2 copper layers, 99 x 108 mm, 38 parts, among them J1 SIGNAL 1, J2 SIGNAL 2, J3 wsout1, J4 wsout2, U3 SN65HVD230, U4 SN65HVD230, U5 ADS1115IDGS

Commit message: awawawaaw jlc
Connections:
- J3 pad 1: WS_FRo -> WS_FLo
- J3 pad 2: WS_FLo -> WS_FRo
- U1 pad 41: WS_FLo -> WS_FRo
- U1 pad 43: WS_FRo -> WS_FLo
Routing:
- net WS_FRo: track 85.7 -> 84.0 mm
- net WS_FLo: track 84.0 -> 85.7 mm
Changed lines of the file:
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@@
 			(layers "*.Cu" "*.Mask")
 			(remove_unused_layers no)
-			(net 109 "WS_FRo")
+			(net 110 "WS_FLo")
 			(pinfunction "Pin_1")
 			(pintype "passive")
@@
 			(layers "*.Cu" "*.Mask")
 			(remove_unused_layers no)
-			(net 110 "WS_FLo")
+			(net 109 "WS_FRo")
 			(pinfunction "Pin_2")
 			(pintype "passive")
@@
 			(layers "*.Cu" "*.Mask")
 			(remove_unused_layers no)
-			(net 110 "WS_FLo")
+			(net 109 "WS_FRo")
 			(pinfunction "PB9")
 			(pintype "input")
@@
 			(layers "*.Cu" "*.Mask")
 			(remove_unused_layers no)
-			(net 109 "WS_FRo")
+			(net 110 "WS_FLo")
 			(pinfunction "PE1")
 			(pintype "input")
@@
 	)
 	(segment
-		(start 130.556 93.98)
-		(end 120.396 93.98)
+		(start 130.556 91.44)
+		(end 124.94 91.44)
 		(width 0.508)
 		(layer "F.Cu")
@@
 	)
 	(segment
-		(start 112 44)
-		(end 113 43)
+		(start 118 44.5)
+		(end 116.5 43)
 		(width 0.508)
 		(layer "F.Cu")
@@
 	)
 	(segment
-		(start 120.396 93.98)
-		(end 112 85.584)
+		(start 124.94 91.44)
+		(end 118 84.5)
 		(width 0.508)
 		(layer "F.Cu")
@@
 	)
 	(segment
-		(start 112 85.584)
-		(end 112 46.25)
+		(start 116.5 43)
+		(end 115.5 43)
 		(width 0.508)
 		(layer "F.Cu")
@@
 	)
 	(segment
-		(start 112 46.25)
-		(end 112 44)
+		(start 118 84.5)
+		(end 118 44.5)
 		(width 0.508)
 		(layer "F.Cu")
@@
 	)
 	(segment
-		(start 110.28 45.72)
-		(end 93.472 45.72)
+		(start 93.472 48.26)
+		(end 112.31369 48.26)
 		(width 0.508)
 		(layer "B.Cu")
@@
 	)
 	(segment
-		(start 113 43)
-		(end 110.28 45.72)
+		(start 112.31369 48.26)
+		(end 115.5 45.07369)
 		(width 0.508)
 		(layer "B.Cu")
@@
 	)
 	(segment
-		(start 130.556 91.44)
-		(end 124.94 91.44)
+		(start 115.5 45.07369)
+		(end 115.5 43)
 		(width 0.508)
-		(layer "F.Cu")
-		(net 110)
+		(layer "B.Cu")
+		(net 109)
 	)
 	(segment
-		(start 124.94 91.44)
-		(end 118 84.5)
+		(start 112 46.25)
+		(end 113 45.25)
 		(width 0.508)
 		(layer "F.Cu")
@@
 	)
 	(segment
-		(start 118 44.5)
-		(end 116.5 43)
+		(start 130.556 93.98)
+		(end 120.396 93.98)
 		(width 0.508)
 		(layer "F.Cu")
@@
 	)
 	(segment
-		(start 116.5 43)
-		(end 115.5 43)
+		(start 120.396 93.98)
+		(end 112 85.584)
 		(width 0.508)
 		(layer "F.Cu")
@@
 	)
 	(segment
-		(start 118 84.5)
-		(end 118 44.5)
+		(start 112 85.584)
+		(end 112 46.25)
 		(width 0.508)
 		(layer "F.Cu")
@@
 	)
 	(segment
-		(start 93.472 48.26)
-		(end 112.31369 48.26)
+		(start 113 45.25)
+		(end 113 43)
 		(width 0.508)
-		(layer "B.Cu")
+		(layer "F.Cu")
 		(net 110)
 	)
 	(segment
-		(start 112.31369 48.26)
-		(end 115.5 45.07369)
+		(start 110.28 45.72)
+		(end 93.472 45.72)
 		(width 0.508)
 		(layer "B.Cu")
@@
 	)
 	(segment
-		(start 115.5 45.07369)
-		(end 115.5 43)
+		(start 110.28 45.72)
+		(end 113 43)
 		(width 0.508)
 		(layer "B.Cu")
