File: Bimasakti BM-13 EVO/PCB/4. Torque Vectoring Board/Torque Vectoring Board.kicad_sch (KiCad schematic)
At the start: 34 parts, among them J1 SIGNAL 1, J2 SIGNAL 2, J3 wsout1, J4 wsout2, U3 SN65HVD230, U4 SN65HVD230, U5 ADS1115IDGS

Commit message: awawawaaw jlc
Connections:
- net WS_FLo: now also J3.1 (Pin_1), U1.43 (PE1); no longer J3.2 (Pin_2), U1.41 (PB9)
- net WS_FRo: now also J3.2 (Pin_2), U1.41 (PB9); no longer J3.1 (Pin_1), U1.43 (PE1)
Changed lines of the file:
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@@
 	(wire
 		(pts
-			(xy 90.17 133.35) (xy 91.44 133.35)
-		)
-		(stroke
-			(width 0)
-			(type default)
-		)
-	)
-	(wire
-		(pts
 			(xy 217.17 80.01) (xy 219.71 80.01)
 		)
@@
 	(wire
 		(pts
+			(xy 256.54 46.99) (xy 256.54 49.53)
+		)
+		(stroke
+			(width 0)
+			(type default)
+		)
+	)
+	(wire
+		(pts
 			(xy 241.3 99.06) (xy 241.3 104.14)
 		)
@@
 	(wire
 		(pts
-			(xy 242.57 64.77) (xy 243.84 64.77)
-		)
-		(stroke
-			(width 0)
-			(type default)
-		)
-	)
-	(wire
-		(pts
 			(xy 134.62 120.65) (xy 139.7 120.65)
 		)
@@
 	(wire
 		(pts
+			(xy 90.17 138.43) (xy 91.44 138.43)
+		)
+		(stroke
+			(width 0)
+			(type default)
+		)
+	)
+	(wire
+		(pts
 			(xy 260.35 46.99) (xy 260.35 49.53)
 		)
@@
 	(wire
 		(pts
+			(xy 242.57 64.77) (xy 243.84 64.77)
+		)
+		(stroke
+			(width 0)
+			(type default)
+		)
+	)
+	(wire
+		(pts
 			(xy 71.12 38.1) (xy 73.66 38.1)
 		)
@@
 	(wire
 		(pts
+			(xy 254 46.99) (xy 254 49.53)
+		)
+		(stroke
+			(width 0)
+			(type default)
+		)
+	)
+	(wire
+		(pts
 			(xy 90.17 102.87) (xy 91.44 102.87)
 		)
@@
 	(wire
 		(pts
-			(xy 256.54 46.99) (xy 256.54 49.53)
-		)
-		(stroke
-			(width 0)
-			(type default)
-		)
-	)
-	(wire
-		(pts
 			(xy 69.85 118.11) (xy 69.85 119.38)
 		)
@@
 	(wire
 		(pts
+			(xy 90.17 133.35) (xy 91.44 133.35)
+		)
+		(stroke
+			(width 0)
+			(type default)
+		)
+	)
+	(wire
+		(pts
 			(xy 200.66 139.7) (xy 209.55 139.7)
 		)
@@
 	(wire
 		(pts
-			(xy 90.17 138.43) (xy 91.44 138.43)
-		)
-		(stroke
-			(width 0)
-			(type default)
-		)
-	)
-	(wire
-		(pts
 			(xy 39.37 83.82) (xy 41.91 83.82)
 		)
@@
 	(wire
 		(pts
+			(xy 242.57 62.23) (xy 243.84 62.23)
+		)
+		(stroke
+			(width 0)
+			(type default)
+		)
+	)
+	(wire
+		(pts
 			(xy 241.3 93.98) (xy 241.3 99.06)
 		)
@@
 	(wire
 		(pts
-			(xy 254 46.99) (xy 254 49.53)
-		)
-		(stroke
-			(width 0)
-			(type default)
-		)
-	)
-	(wire
-		(pts
 			(xy 148.59 90.17) (xy 154.94 90.17)
 		)
@@
 	(wire
 		(pts
-			(xy 242.57 62.23) (xy 243.84 62.23)
-		)
-		(stroke
-			(width 0)
-			(type default)
-		)
-	)
-	(wire
-		(pts
 			(xy 46.99 139.7) (xy 46.99 142.24)
 		)
@@
 	(global_label "WS_FRo"
 		(shape input)
-		(at 254 49.53 270)
+		(at 256.54 49.53 270)
 		(fields_autoplaced yes)
 		(effects
@@
 		)
 		(property "Intersheetrefs" "${INTERSHEET_REFS}"
-			(at 254 59.6513 90)
+			(at 256.54 59.6513 90)
 			(effects
 				(font
@@
 	(global_label "WS_FLo"
 		(shape input)
-		(at 90.17 133.35 180)
+		(at 90.17 138.43 180)
 		(fields_autoplaced yes)
 		(effects
@@
 		)
 		(property "Intersheetrefs" "${INTERSHEET_REFS}"
-			(at 80.2906 133.35 0)
+			(at 80.2906 138.43 0)
 			(effects
 				(font
@@
 	(global_label "WS_FLo"
 		(shape input)
-		(at 256.54 49.53 270)
+		(at 254 49.53 270)
 		(fields_autoplaced yes)
 		(effects
@@
 		)
 		(property "Intersheetrefs" "${INTERSHEET_REFS}"
-			(at 256.54 59.4094 90)
+			(at 254 59.4094 90)
 			(effects
 				(font
@@
 	(global_label "WS_FRo"
 		(shape input)
-		(at 90.17 138.43 180)
+		(at 90.17 133.35 180)
 		(fields_autoplaced yes)
 		(effects
@@
 		)
 		(property "Intersheetrefs" "${INTERSHEET_REFS}"
-			(at 80.0487 138.43 0)
+			(at 80.0487 133.35 0)
 			(effects
 				(font
