File: Bimasakti BM-13 EVO/PCB/8. Telemetry/Telemetry V.3 BM13 EVO Hy.kicad_pcb (KiCad board)
At the start: 2 copper layers, 83.5 x 70 mm, 28 parts, among them J1 MSD-4-A, J2 CON INT/32, J4 Conn_01x16_Pin, U1 ESP32-DEVKIT-V1, U2 74LVC125APW_118, U3 DS3231SN_

Commit message: awawawaaw jlc
Routing:
- net GND: vias 62 -> 68
Changed lines of the file:
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@@
 			(outputformat 1)
 			(mirror no)
-			(drillshape 1)
+			(drillshape 0)
 			(scaleselection 1)
-			(outputdirectory "")
+			(outputdirectory "JLC/")
 		)
 	)
@@
 	)
 	(via
+		(at 90.25 64)
+		(size 0.6)
+		(drill 0.3)
+		(layers "F.Cu" "B.Cu")
+		(free yes)
+		(net 1)
+	)
+	(via
 		(at 113.4 55.4)
 		(size 0.6)
@@
 	)
 	(via
+		(at 91.25 64)
+		(size 0.6)
+		(drill 0.3)
+		(layers "F.Cu" "B.Cu")
+		(free yes)
+		(net 1)
+	)
+	(via
 		(at 112.6 53)
 		(size 0.6)
@@
 	)
 	(via
+		(at 92.25 61.5)
+		(size 0.6)
+		(drill 0.3)
+		(layers "F.Cu" "B.Cu")
+		(free yes)
+		(net 1)
+	)
+	(via
 		(at 117.4 53)
 		(size 0.6)
@@
 	)
 	(via
+		(at 92.25 64)
+		(size 0.6)
+		(drill 0.3)
+		(layers "F.Cu" "B.Cu")
+		(free yes)
+		(net 1)
+	)
+	(via
 		(at 113 80.5)
 		(size 0.5)
@@
 	)
 	(via
+		(at 90.25 61.5)
+		(size 0.6)
+		(drill 0.3)
+		(layers "F.Cu" "B.Cu")
+		(free yes)
+		(net 1)
+	)
+	(via
 		(at 99 80)
 		(size 0.6)
@@
 		(layers "F.Cu" "B.Cu")
 		(free yes)
+		(net 1)
+	)
+	(via
+		(at 91.25 61.5)
+		(size 0.6)
+		(drill 0.3)
+		(layers "F.Cu" "B.Cu")
+		(free yes)
